Commit message: control period of plugin to 0.001 and updated traction torque

File: rbcar_description/urdf/bases/rbcar_base.gazebo.xacro (robot description, xacro)
@@ -7,5 +7,6 @@
         <robotNamespace>/rbcar</robotNamespace>
         <robotParam>robot_description</robotParam>
-        <controlPeriod>0.003</controlPeriod>
+        <!-- controlPeriod>0.003</controlPeriod -->
+        <controlPeriod>0.001</controlPeriod>
 	    <robotSimType>gazebo_ros_control/DefaultRobotHWSim</robotSimType>
       </plugin>

File: rbcar_description/urdf/wheels/suspension_wheel.urdf.xacro (robot description, xacro)
@@ -31,5 +31,6 @@
        (calculating this way, it should be divided by 2 if 2 motors are used)
        axle_eff_limit = 204.95 / 2 N m = ~102.5 -->
-  <xacro:property name="axle_eff_limit" value="102.5"/>
+  <!-- xacro:property name="axle_eff_limit" value="102.5"/ -->
+  <xacro:property name="axle_eff_limit" value="204.95"/>
   <!-- max_speed = 33 Km/h = 9.17 m/s
        axle_vel_limit = (2 * pi) * (max_speed / (pi * tire_dia)) =  39.02 rad/s -->
