Commit message: updated description of the robot

File: rbcar_description/urdf/bases/rbcar_base_v2.urdf.xacro (robot description, xacro)
@@ -41,13 +41,13 @@
       </inertial>
       <visual>
-        <origin xyz="0 0 0" rpy="0 0 0" />
+        <origin xyz="0 0 0.175" rpy="0 0 0" />
         <xacro:if value="${hq}">
           <geometry>
-            <mesh filename="package://rbcar_description/meshes/bases/rbcar_chassis_v2.STL"/>
+            <mesh filename="package://rbcar_description/meshes/bases/rbcar_chassis_v2.stl"/>
           </geometry>
         </xacro:if>
         <xacro:unless value="${hq}">
           <geometry>
-            <mesh filename="package://rbcar_description/meshes/bases/rbcar_chassis_v2.STL"/>
+            <mesh filename="package://rbcar_description/meshes/bases/rbcar_chassis_v2.stl"/>
           </geometry>
         </xacro:unless>
@@ -59,5 +59,5 @@
         <origin xyz="0 0 0" rpy="0 0 0 " />
         <geometry>
-          <mesh filename="package://rbcar_description/meshes/bases/rbcar_chassis_v2.STL"/>
+          <mesh filename="package://rbcar_description/meshes/bases/rbcar_chassis_v2.stl"/>
         </geometry>
       </collision>

File: rbcar_description/urdf/wheels/suspension_wheel_v2.urdf (copia).xacro (robot description, xacro)
@@ -1,5 +1,4 @@
 <?xml version="1.0"?>
-<robot name="wheel"
-  xmlns:xacro="http://wiki.ros.org/xacro">
+<robot name="wheel" xmlns:xacro="http://wiki.ros.org/xacro">
   <!-- hub_dia and tire_dia are the diameters of the hub and tire,
        respectively. hex_hub_depth is the distance that the hex hub is
@@ -10,21 +9,17 @@
   <xacro:property name="tire_dia" value="0.440"/>
   <xacro:property name="tire_width" value="0.195"/>
-  <xacro:property name="hex_hub_depth" value="0.120"/>
-  <!-- or +0.072 -->
-  <xacro:property name="wheel_mass" value="8.0"/>
-  <!-- check -->
+  <xacro:property name="hex_hub_depth" value="0.120"/> <!-- or +0.072 -->
+  <xacro:property name="wheel_mass" value="8.0"/>   <!-- check -->
   <!-- hex_hub_dist is the distance between left and right hex hubs when
        the shock absorbers are fully extended. axle_length is the distance
        from a U joint to the corresponding hex hub. wheel_travel is the
        vertical wheel travel. -->
-  <xacro:property name="wheelbase" value="1.63"/>
-  <xacro:property name="hex_hub_dist" value="0.9191"/>
-  <!-- 1.127 0.742 0.900 check -->
+  <xacro:property name="wheelbase" value="2.5"/>
+  <xacro:property name="hex_hub_dist" value="0.9191"/>  <!-- 1.127 0.742 0.900 check -->
   <xacro:property name="axle_length" value="0.120"/>
   <xacro:property name="wheel_travel" value="0.1"/>
   <xacro:property name="shock_z_offset" value="0.05"/>
   <!-- Degree-to-radian conversions -->
-  <xacro:property name="degrees_34" value="0.60822457"/>
-  <!-- this is used as the limit of the steering of the wheels -->
+  <xacro:property name="degrees_34" value="0.60822457"/> <!-- this is used as the limit of the steering of the wheels -->
   <xacro:property name="degrees_45" value="0.785398163"/>
   <xacro:property name="degrees_90" value="1.57079633"/>
@@ -48,17 +43,20 @@
   <!-- Servo_stall_torque of the direction axis in Nm. servo_no_load_speed is
        measured in rad/s. -->
-  <xacro:property name="servo_stall_torque" value="50"/>
-  <!-- check -->
-  <xacro:property name="servo_no_load_speed" value="25"/>
-  <!-- check -->
+  <xacro:property name="servo_stall_torque" value="50"/>  <!-- check -->
+  <xacro:property name="servo_no_load_speed" value="25"/> <!-- check -->
   <!-- Inertia of a thick-walled cylindrical tube with open ends. Height is
        measured along the z axis, which is the tube's axis. inner_rad and
        outer_rad are the tube's inner and outer radii, respectively. -->
-  <xacro:macro name="thick_walled_tube_inertial" params="inner_rad outer_rad height mass">
+  <xacro:macro name="thick_walled_tube_inertial"
+               params="inner_rad outer_rad height mass">
     <inertial>
       <mass value="${mass}"/>
       <inertia ixx="${(1 / 12) * mass * (3 * (inner_rad * inner_rad +
-                    outer_rad * outer_rad) + height * height)}" ixy="0" ixz="0" iyy="${(1 / 12) * mass * (3 * (inner_rad * inner_rad +
-                    outer_rad * outer_rad) + height * height)}" iyz="0" izz="${mass * (inner_rad * inner_rad +
+                    outer_rad * outer_rad) + height * height)}"
+               ixy="0" ixz="0"
+               iyy="${(1 / 12) * mass * (3 * (inner_rad * inner_rad +
+                    outer_rad * outer_rad) + height * height)}"
+               iyz="0"
+               izz="${mass * (inner_rad * inner_rad +
                     outer_rad * outer_rad) / 2}"/>
     </inertial>
@@ -73,6 +71,7 @@
   </xacro:macro>
   <!-- Shock absorber -->
-  <xacro:macro name="shock" params="lr_prefix fr_prefix lr_reflect fr_reflect child parent prefix:=^''">
-    <joint name="${prefix}${lr_prefix}_${fr_prefix}_shock" type="prismatic">
+  <xacro:macro name="shock"
+               params="lr_prefix fr_prefix lr_reflect fr_reflect child parent prefix">
+    <joint name="${robot_prefix}_${lr_prefix}_${fr_prefix}_shock" type="prismatic">
       <parent link="${parent}"/>
       <child link="${child}"/>
@@ -87,13 +86,14 @@
                    ${(wheel_travel / 2) - shock_z_offset}"/>
       <axis xyz="0 0 -1"/>
-      <limit lower="${-wheel_travel / 2}" upper="${wheel_travel / 2}" effort="${shock_eff_limit}" velocity="${shock_vel_limit}"/>
+      <limit lower="${-wheel_travel / 2}" upper="${wheel_travel / 2}"
+             effort="${shock_eff_limit}" velocity="${shock_vel_limit}"/>
       <joint_properties damping="${suspension_joint_damping}" friction="${suspension_joint_friction}"/>
     </joint>
-    <transmission name="${prefix}${lr_prefix}_${fr_prefix}_shock_trans">
+    <transmission name="${robot_prefix}_${lr_prefix}_${fr_prefix}_shock_trans">
       <type>transmission_interface/SimpleTransmission</type>
-      <joint name="${prefix}${lr_prefix}_${fr_prefix}_shock">
+      <joint name="${robot_prefix}_${lr_prefix}_${fr_prefix}_shock">
         <hardwareInterface>hardware_interface/EffortJointInterface</hardwareInterface>
       </joint>
-      <actuator name="${prefix}${lr_prefix}_${fr_prefix}_shock_act">
+      <actuator name="${robot_prefix}_${lr_prefix}_${fr_prefix}_shock_act">
         <mechanicalReduction>1</mechanicalReduction>
       </actuator>
@@ -101,7 +101,7 @@
   </xacro:macro>
   <!-- The "wheel" macro defines an axle carrier, axle, and wheel. -->
-  <xacro:macro name="wheel" params="lr_prefix fr_prefix lr_reflect prefix:=^''">
-    <link name="${prefix}${lr_prefix}_${fr_prefix}_axle_carrier">
-      <!-- visual>
+  <xacro:macro name="wheel" params="lr_prefix fr_prefix lr_reflect">
+    <link name="${lr_prefix}_${fr_prefix}_axle_carrier">
+	  <!-- visual>
         <origin xyz="0 0 0"/>
         <geometry>
@@ -119,7 +119,7 @@
     <!-- The left and right axles have the same axis so that identical
          rotation values cause the wheels to rotate in the same direction. -->
-    <joint name="${prefix}${lr_prefix}_${fr_prefix}_axle" type="continuous">
-      <parent link="${prefix}${lr_prefix}_${fr_prefix}_axle_carrier"/>
-      <child link="${prefix}${lr_prefix}_${fr_prefix}_wheel"/>
+    <joint name="${robot_prefix}_${lr_prefix}_${fr_prefix}_axle" type="continuous">
+      <parent link="${robot_prefix}_${lr_prefix}_${fr_prefix}_axle_carrier"/>
+      <child link="${robot_prefix}_${lr_prefix}_${fr_prefix}_wheel"/>
       <origin rpy="${degrees_90} 0 ${degrees_180}"/>
       <axis xyz="0 0 1"/>
@@ -127,18 +127,18 @@
       <joint_properties damping="${wheel_joint_damping}" friction="${wheel_joint_friction}"/>
     </joint>
-    <transmission name="${prefix}${lr_prefix}_${fr_prefix}_axle_trans">
+    <transmission name="${robot_prefix}_${lr_prefix}_${fr_prefix}_axle_trans">
       <type>transmission_interface/SimpleTransmission</type>
-      <joint name="${prefix}${lr_prefix}_${fr_prefix}_axle">
+      <joint name="${robot_prefix}_${lr_prefix}_${fr_prefix}_axle">
         <!-- hardwareInterface>hardware_interface/EffortJointInterface</hardwareInterface -->
         <hardwareInterface>hardware_interface/VelocityJointInterface</hardwareInterface>
       </joint>
-      <actuator name="${prefix}${lr_prefix}_${fr_prefix}_axle_act">
+      <actuator name="${robot_prefix}_${lr_prefix}_${fr_prefix}_axle_act">
         <mechanicalReduction>1</mechanicalReduction>
       </actuator>
     </transmission>
-    <gazebo reference="${prefix}${lr_prefix}_${fr_prefix}_axle_carrier">
+    <gazebo reference="${robot_prefix}_${lr_prefix}_${fr_prefix}_axle_carrier">
       <material>Gazebo/Black</material>
     </gazebo>
-    <link name="${prefix}${lr_prefix}_${fr_prefix}_wheel">
+    <link name="${robot_prefix}_${lr_prefix}_${fr_prefix}_wheel">
       <visual>
         <xacro:if value="${lr_prefix=='left'}">
@@ -165,7 +165,9 @@
         </geometry>
       </collision>
-      <xacro:thick_walled_tube_inertial inner_rad="${hub_dia / 2}" outer_rad="${tire_dia / 2}" height="${tire_width}" mass="${wheel_mass}"/>
+      <xacro:thick_walled_tube_inertial
+          inner_rad="${hub_dia / 2}" outer_rad="${tire_dia / 2}"
+          height="${tire_width}" mass="${wheel_mass}"/>
     </link>
-    <gazebo reference="${prefix}${lr_prefix}_${fr_prefix}_wheel">
+    <gazebo reference="${robot_prefix}_${lr_prefix}_${fr_prefix}_wheel">
       <material>Gazebo/Black</material>
     </gazebo>
@@ -173,8 +175,11 @@
   <!-- xacro:macro name="rubber_wheel" params="name parent *origin reflect hq" -->
   <!-- Front wheel -->
-  <xacro:macro name="front_wheel" params="lr_prefix fr_prefix lr_reflect fr_reflect parent prefix:=^''">
-    <xacro:shock lr_prefix="${lr_prefix}" fr_prefix="${fr_prefix}" lr_reflect="${lr_reflect}" fr_reflect="${fr_reflect}" child="${prefix}${lr_prefix}_steering_link" parent="${parent}" prefix="${prefix}"/>
-    <link name="${prefix}${lr_prefix}_steering_link">
-      <!-- visual>
+  <xacro:macro name="front_wheel"
+               params="lr_prefix fr_prefix lr_reflect fr_reflect parent">
+    <xacro:shock lr_prefix="${lr_prefix}" fr_prefix="${fr_prefix}"
+                 lr_reflect="${lr_reflect}" fr_reflect="${fr_reflect}"
+                 child="${robot_prefix}_${lr_prefix}_steering_link" parent="${parent}"/>
+    <link name="${lr_prefix}_steering_link">
+	  <!-- visual>
 		<origin xyz="0 0 0"/>
         <geometry>
@@ -190,34 +195,41 @@
       <xacro:null_inertial/>
     </link>
-    <joint name="${prefix}${lr_prefix}_steering_joint" type="revolute">
-      <parent link="${prefix}${lr_prefix}_steering_link"/>
-      <child link="${prefix}${lr_prefix}_${fr_prefix}_axle_carrier"/>
+    <joint name="${robot_prefix}_${lr_prefix}_steering_joint" type="revolute">
+      <parent link="${robot_prefix}_${lr_prefix}_steering_link"/>
+      <child link="${robot_prefix}_${lr_prefix}_${fr_prefix}_axle_carrier"/>
       <axis xyz="0 0 1"/>
-      <xacro:if value="${lr_reflect == 1}">        <!-- this applies if we are setting the left wheel -->
-        <limit lower="${-degrees_34}" upper="${degrees_45}" effort="${servo_stall_torque}" velocity="${servo_no_load_speed}"/>
-      </xacro:if>
-      <xacro:unless value="${lr_reflect == 1}">        <!-- this applies if we are setting the right wheel -->
-        <limit lower="${-degrees_45}" upper="${degrees_34}" effort="${servo_stall_torque}" velocity="${servo_no_load_speed}"/>
+      <xacro:if value="${lr_reflect == 1}"> <!-- this applies if we are setting the left wheel -->
+        <limit lower="${-degrees_34}" upper="${degrees_45}"
+             effort="${servo_stall_torque}" velocity="${servo_no_load_speed}"/>
+        </xacro:if>
+      <xacro:unless value="${lr_reflect == 1}"> <!-- this applies if we are setting the right wheel -->
+        <limit lower="${-degrees_45}" upper="${degrees_34}"
+             effort="${servo_stall_torque}" velocity="${servo_no_load_speed}"/>
       </xacro:unless>
     </joint>
-    <transmission name="${prefix}${lr_prefix}_steering_trans">
+    <transmission name="${robot_prefix}_${lr_prefix}_steering_trans">
       <type>transmission_interface/SimpleTransmission</type>
-      <joint name="${prefix}${lr_prefix}_steering_joint">
+      <joint name="${robot_prefix}_${lr_prefix}_steering_joint">
         <!--<hardwareInterface>hardware_interface/EffortJointInterface</hardwareInterface>-->
         <hardwareInterface>hardware_interface/PositionJointInterface</hardwareInterface>
       </joint>
-      <actuator name="${prefix}${lr_prefix}_steering_act">
+      <actuator name="${robot_prefix}_${lr_prefix}_steering_act">
         <mechanicalReduction>1</mechanicalReduction>
       </actuator>
     </transmission>
-    <gazebo reference="${prefix}${lr_prefix}_steering_link">
+    <gazebo reference="${robot_prefix}_${lr_prefix}_steering_link">
       <material>Gazebo/Black</material>
     </gazebo>
-    <xacro:wheel lr_prefix="${lr_prefix}" fr_prefix="${fr_prefix}" lr_reflect="${lr_reflect}" prefix="${prefix}"/>
+    <xacro:wheel lr_prefix="${lr_prefix}" fr_prefix="${fr_prefix}"
+                 lr_reflect="${lr_reflect}"/>
   </xacro:macro>
   <!-- Rear wheel -->
-  <xacro:macro name="rear_wheel" params="lr_prefix fr_prefix lr_reflect fr_reflect parent prefix:=^''">
-    <xacro:shock lr_prefix="${lr_prefix}" fr_prefix="${fr_prefix}" lr_reflect="${lr_reflect}" fr_reflect="${fr_reflect}" child="${prefix}${lr_prefix}_${fr_prefix}_axle_carrier" parent="${parent}" prefix="${prefix}"/>
-    <xacro:wheel lr_prefix="${lr_prefix}" fr_prefix="${fr_prefix}" lr_reflect="${lr_reflect}" prefix="${prefix}"/>
-  </xacro:macro>
-</robot>
+  <xacro:macro name="rear_wheel"
+               params="lr_prefix fr_prefix lr_reflect fr_reflect parent">
+    <xacro:shock lr_prefix="${lr_prefix}" fr_prefix="${fr_prefix}"
+                 lr_reflect="${lr_reflect}" fr_reflect="${fr_reflect}"
+                 child="${robot_prefix}_${lr_prefix}_${fr_prefix}_axle_carrier" parent="${parent}"/>
+    <xacro:wheel lr_prefix="${lr_prefix}" fr_prefix="${fr_prefix}"
+                 lr_reflect="${lr_reflect}"/>
+  </xacro:macro>
+ </robot>

Commit message: changed z of the rbcar_base

File: rbcar_description/urdf/bases/rbcar_base_v2.urdf.xacro (robot description, xacro)
@@ -57,5 +57,5 @@
       </visual>
       <collision>
-        <origin xyz="0 0 0" rpy="0 0 0 " />
+        <origin xyz="0 0 0.175" rpy="0 0 0 " />
         <geometry>
           <mesh filename="package://rbcar_description/meshes/bases/rbcar_chassis_v2.stl"/>

Commit message: added wheelbase param

File: rbcar_description/urdf/bases/rbcar_base_v2.urdf.xacro (robot description, xacro)
@@ -3,5 +3,5 @@
   xmlns:xacro="http://www.ros.org/wiki/xacro">
   <xacro:include filename="$(find rbcar_description)/urdf/bases/rbcar_base.gazebo.xacro" />
-  <xacro:macro name="rbcar_base" params="name publish_bf hq prefix:=^''">
+  <xacro:macro name="rbcar_base" params="name publish_bf hq prefix:=^'' wheelbase:=^'1.63'">
     <!-- Robot mechanical and motor parameters -->
     <xacro:property name="PI" value="3.1415926535897931"/>
@@ -37,9 +37,9 @@
       <inertial>
         <mass value="125.0" />
-        <origin xyz="0 0 0" />
+        <origin xyz="${wheelbase/2.0} 0 0" />
         <inertia ixx="1.391" ixy="0.004" ixz="0.0" iyy="6.853" iyz="0.0" izz="6.125" />
       </inertial>
       <visual>
-        <origin xyz="0 0 0.175" rpy="0 0 0" />
+        <origin xyz="${wheelbase/2.0} 0 0.175" rpy="0 0 0" />
         <xacro:if value="${hq}">
           <geometry>
@@ -57,5 +57,5 @@
       </visual>
       <collision>
-        <origin xyz="0 0 0.175" rpy="0 0 0 " />
+        <origin xyz="${wheelbase/2.0} 0 0.175" rpy="0 0 0 " />
         <geometry>
           <mesh filename="package://rbcar_description/meshes/bases/rbcar_chassis_v2.stl"/>
