Commit message: corrected ranges of hokuyo3d and added measurement tf

File: rbcar_description/urdf/bases/rbcar_base.urdf.xacro (robot description, xacro)
@@ -25,6 +25,5 @@
     </link>
     <joint name="base_footprint_joint" type="fixed">
-      <!-- origin xyz="0 0 ${wheel_radius}" rpy="0 0 0" / --> <!-- ${wheel_radius} property must be defined inside wheel description -->
-      <origin xyz="0 0 ${tire_dia / 2}" rpy="0 0 0" /> <!-- ${wheel_radius} property must be defined inside wheel description -->
+      <origin xyz="0 0 0.150" rpy="0 0 0" />  <!-- height is the clearance -->
       <parent link="base_footprint"/>
       <child link="base_link" />

File: rbcar_description/urdf/sensors/hokuyo3d.urdf.xacro (robot description, xacro)
@@ -2,10 +2,10 @@
 <robot name="sensor_hokuyo3d" xmlns:xacro="http://ros.org/wiki/xacro">
   <xacro:macro name="sensor_hokuyo3d" params="name parent *origin">
-    <joint name="${name}_laser_joint" type="fixed">
+    <joint name="${name}_laser_fix_joint" type="fixed">
       <insert_block name="origin" />
       <parent link="${parent}"/>
-      <child link="${name}_laser_link"/>
+      <child link="${name}_laser_fix_link"/>
 	</joint>
-	<link name="${name}_laser_link">
+	<link name="${name}_laser_fix_link">
 		<collision>
 			<origin xyz="0 0 0" rpy="0 0 0"/>
@@ -26,4 +26,11 @@
 		</inertial>
 	</link>
+	<link name="${name}_laser_link">
+	</link>
+    <joint name="${name}_laser_joint" type="fixed">
+      <parent link="${name}_laser_fix_link"/>
+      <child link="${name}_laser_link"/>
+      <origin xyz="0.08 0 0.08" rpy="0 0 0"/>
+	</joint>
 	<!-- Hokuyo sensor for simulation -->
 	<sensor_hokuyo3d_gazebo/>
@@ -47,6 +54,6 @@
                             <samples>74</samples>
                             <resolution>1.0</resolution>
-                            <min_angle>-0.0872664626</min_angle>
-                            <max_angle>0.610865238</max_angle>
+                            <min_angle>-0.610865238</min_angle>
+                            <max_angle>0.0872664626</max_angle>
                         </vertical>
 					</scan>

Commit message: description: adjusting wheels position

File: rbcar_description/urdf/bases/rbcar_base.urdf.xacro (robot description, xacro)
@@ -6,4 +6,5 @@
   <xacro:property name="PI" value="3.1415926535897931"/>
   <xacro:property name="wheel_width" value="0.175" />
+  <xacro:property name="clearance" value="${tire_dia/2.0}" />
   <!-- BASE FOOTPRINT -->
   <xacro:if value="${publish_bf}">
@@ -25,5 +26,5 @@
     </link>
     <joint name="base_footprint_joint" type="fixed">
-      <origin xyz="0 0 0.235" rpy="0 0 0" />  <!-- height is the clearance -->
+      <origin xyz="0 0 ${clearance}" rpy="0 0 0" />  <!-- height is the clearance -->
       <parent link="base_footprint"/>
       <child link="base_link" />

File: rbcar_description/urdf/wheels/suspension_wheel.urdf.xacro (robot description, xacro)
@@ -16,5 +16,5 @@
        vertical wheel travel. -->
   <xacro:property name="wheelbase" value="1.650"/>
-  <xacro:property name="hex_hub_dist" value="0.900"/>  <!-- 1.127 0.742 check -->
+  <xacro:property name="hex_hub_dist" value="0.900"/>  <!-- 1.127 0.742 0.900 check -->
   <xacro:property name="axle_length" value="0.120"/>
   <xacro:property name="wheel_travel" value="0.1"/>
@@ -77,5 +77,6 @@
       <origin xyz="${fr_reflect * wheelbase / 2}
                    ${lr_reflect * ((hex_hub_dist / 2) - axle_length)}
-                   ${(wheel_travel / 2) - shock_z_offset}"/>
+                   ${-wheel_travel}"/>
+                  <!-- ${(wheel_travel / 2) - shock_z_offset}"/-->
       <axis xyz="0 0 -1"/>
       <limit lower="${-wheel_travel / 2}" upper="${wheel_travel / 2}"

Commit message: bug fixed

File: rbcar_description/urdf/bases/rbcar_base.urdf.xacro (robot description, xacro)
@@ -57,5 +57,5 @@
        <origin xyz="0.917 0 0" rpy="0 0 0 " />
        <geometry>
-         <mesh filename="package://rbcar_description/meshes/bases/roborder_chassis.stl"/>
+         <mesh filename="package://rbcar_description/meshes/bases/rbcar_chassis.stl"/>
        </geometry>
     </collision>

Commit message: 3d model hq updated

File: rbcar_description/urdf/bases/rbcar_base.urdf.xacro (robot description, xacro)
@@ -42,5 +42,5 @@
        <xacro:if value="${hq}">
        <geometry>
-	     <mesh filename="package://rbcar_description/meshes/bases/rbcar_chassis.stl"/>
+	     <mesh filename="package://rbcar_description/meshes/bases/rbcar_chassis_hq.stl"/>
        </geometry>
        </xacro:if>

Commit message: aded default empty value for prefix arg

File: rbcar_description/urdf/bases/rbcar_base.urdf.xacro (robot description, xacro)
@@ -2,5 +2,5 @@
 <robot name="rbcar" xmlns:xacro="http://wiki.ros.org/xacro">
   <xacro:include filename="$(find rbcar_description)/urdf/bases/rbcar_base.gazebo.xacro" />
-  <xacro:macro name="rbcar_base" params="prefix name publish_bf hq">
+  <xacro:macro name="rbcar_base" params="prefix:='' name publish_bf hq">
   <!-- Robot mechanical and motor parameters -->
   <xacro:property name="PI" value="3.1415926535897931"/>

Commit message: minor adjustment

File: rbcar_description/urdf/bases/rbcar_base.urdf.xacro (robot description, xacro)
@@ -6,5 +6,5 @@
   <xacro:property name="PI" value="3.1415926535897931"/>
   <xacro:property name="wheel_width" value="0.317" />
-  <xacro:property name="clearance" value="${tire_dia/2.0}" />
+  <xacro:property name="clearance" value="0.31" />
   <!-- BASE FOOTPRINT -->
   <xacro:if value="${publish_bf}">
