Commit message: changed hw interface to VelocityJointInterface for traction, added damping and friction to axle and suspension

File: rbcar_description/urdf/wheels/suspension_wheel.urdf.xacro (robot description, xacro)
@@ -27,4 +27,8 @@
   <xacro:property name="shock_eff_limit" value="100"/>
   <xacro:property name="shock_vel_limit" value="1000"/>
+  <xacro:property name="wheel_joint_damping" value="0.2" />
+  <xacro:property name="wheel_joint_friction" value="0.7" />
+  <xacro:property name="suspension_joint_damping" value="0.2" />
+  <xacro:property name="suspension_joint_friction" value="0.7" />
   <!-- axle eff limit = 2 * stall_torque
        as a function of the max gradient (15%) with overall max payload (600Kg) * wheel_radius
@@ -77,4 +81,5 @@
       <limit lower="${-wheel_travel / 2}" upper="${wheel_travel / 2}"
              effort="${shock_eff_limit}" velocity="${shock_vel_limit}"/>
+      <joint_properties damping="${suspension_joint_damping}" friction="{suspension_joint_friction}"/>
     </joint>
     <transmission name="${lr_prefix}_${fr_prefix}_shock_trans">
@@ -84,7 +89,4 @@
       </joint>
       <actuator name="${lr_prefix}_${fr_prefix}_shock_act">
-        <!-- This hardwareInterface element exists for compatibility
-             with ROS Hydro. -->
-        <hardwareInterface>EffortJointInterface</hardwareInterface>
         <mechanicalReduction>1</mechanicalReduction>
       </actuator>
@@ -116,14 +118,13 @@
       <axis xyz="0 0 -1"/>
       <limit effort="${axle_eff_limit}" velocity="${axle_vel_limit}"/>
+      <joint_properties damping="${wheel_joint_damping}" friction="{wheel_joint_friction}"/>
     </joint>
     <transmission name="${lr_prefix}_${fr_prefix}_axle_trans">
       <type>transmission_interface/SimpleTransmission</type>
       <joint name="${lr_prefix}_${fr_prefix}_axle">
-        <hardwareInterface>EffortJointInterface</hardwareInterface>
+        <!-- hardwareInterface>EffortJointInterface</hardwareInterface -->
+        <hardwareInterface>VelocityJointInterface</hardwareInterface>
       </joint>
       <actuator name="${lr_prefix}_${fr_prefix}_axle_act">
-        <!-- This hardwareInterface element exists for compatibility
-             with ROS Hydro. -->
-        <hardwareInterface>EffortJointInterface</hardwareInterface>
         <mechanicalReduction>1</mechanicalReduction>
       </actuator>
@@ -193,7 +194,4 @@
       </joint>
       <actuator name="${lr_prefix}_steering_act">
-        <!-- This hardwareInterface element exists for compatibility
-             with ROS Hydro. -->
-        <hardwareInterface>EffortJointInterface</hardwareInterface>
         <mechanicalReduction>1</mechanicalReduction>
       </actuator>
