Commit message: different steering limits for inner/outer wheel (34/45 degrees)

File: rbcar_description/urdf/wheels/suspension_wheel_v2.urdf.xacro (robot description, xacro)
@@ -21,4 +21,5 @@
   <xacro:property name="shock_z_offset" value="0.05"/>
   <!-- Degree-to-radian conversions -->
+  <xacro:property name="degrees_34" value="0.60822457"/> <!-- this is used as the limit of the steering of the wheels -->
   <xacro:property name="degrees_45" value="0.785398163"/>
   <xacro:property name="degrees_90" value="1.57079633"/>
@@ -199,6 +200,12 @@
       <child link="${lr_prefix}_${fr_prefix}_axle_carrier"/>
       <axis xyz="0 0 1"/>
-      <limit lower="${-degrees_45}" upper="${degrees_45}"
+      <xacro:if value="${lr_reflect == 1}"> <!-- this applies if we are setting the left wheel -->
+        <limit lower="${-degrees_34}" upper="${degrees_45}"
              effort="${servo_stall_torque}" velocity="${servo_no_load_speed}"/>
+        </xacro:if>
+      <xacro:unless value="${lr_reflect == 1}"> <!-- this applies if we are setting the right wheel -->
+        <limit lower="${-degrees_45}" upper="${degrees_34}"
+             effort="${servo_stall_torque}" velocity="${servo_no_load_speed}"/>
+      </xacro:unless>
     </joint>
     <transmission name="${lr_prefix}_steering_trans">

Commit message: fixed up the position of the wheels

File: rbcar_description/urdf/wheels/suspension_wheel_v2.urdf.xacro (robot description, xacro)
@@ -82,5 +82,5 @@
         <xacro:property name="hex_hub_dist" value="1.2385"/>
       </xacro:if>
-      <origin xyz="${fr_reflect * wheelbase / 2 + 0.917}
+      <origin xyz="${fr_reflect * wheelbase / 2}
                    ${lr_reflect * ((hex_hub_dist / 2) - axle_length)}
                    ${(wheel_travel / 2) - shock_z_offset}"/>
@@ -145,10 +145,10 @@
           <origin xyz="0
                        0
-                       ${lr_reflect * (axle_length - (tire_width / 2 - hex_hub_depth))}" rpy = "${degrees_90} 0 ${degrees_180}"/>
+                       ${lr_reflect * (axle_length - (tire_width / 2 - hex_hub_depth))}" rpy="0 0 0"/>
         </xacro:if>
         <xacro:if value="${lr_prefix=='right'}">
           <origin xyz="0
                        0
-                       ${lr_reflect * (axle_length - (tire_width / 2 - hex_hub_depth))}" rpy = "-${degrees_90} 0 ${degrees_180}"/>
+                       ${lr_reflect * (axle_length - (tire_width / 2 - hex_hub_depth))}" rpy="0 0 ${degrees_180}"/>
         </xacro:if>
         <geometry>

Commit message: added wheelbase param

File: rbcar_description/urdf/wheels/suspension_wheel_v2.urdf.xacro (robot description, xacro)
@@ -83,5 +83,5 @@
         <xacro:property name="hex_hub_dist" value="1.2385"/>
       </xacro:if>
-      <origin xyz="${fr_reflect * wheelbase / 2}
+      <origin xyz="${fr_reflect * wheelbase / 2 + wheelbase/2}
                    ${lr_reflect * ((hex_hub_dist / 2) - axle_length)}
                    ${(wheel_travel / 2) - shock_z_offset}"/>
