Commit message: Make rear axle (virtual joint) invisible.

File: rbcar_description/urdf/wheels/rear_axle.urdf.xacro (robot description, xacro)
@@ -22,5 +22,5 @@
     </transmission>
     <link name="${prefix}">
-      <visual>
+      <!-- <visual>
         <origin xyz="0 0 0"/>
         <geometry>
@@ -28,5 +28,5 @@
         </geometry>
         <material name="tire_mat"/>
-      </visual>
+      </visual> -->
       <collision>
         <origin xyz="0 0 0"/>
