Commit message: added robot description ezgo model

File: rbcar_description/robots/rbcar_ezgo.urdf.xacro (robot description, xacro)
@@ -6,9 +6,9 @@
 	<!-- First we import all posible elements defined in the urdf.xacro files. All these elements are defined as macro:xacros -->
 	<!-- Import Robotnik CAR base elements -->
-	<xacro:include filename="$(find rbcar_description)/urdf/bases/rbcar_base.urdf.xacro" />
+	<xacro:include filename="$(find rbcar_description)/urdf/bases/rbcar_base_ezgo.urdf.xacro" />
 	<!-- Import Robotnik CAR wheels -->
-    <xacro:property name="wheelbase" value="1.650"/>
-    <xacro:property name="hex_hub_dist" value="0.900"/>
-    <xacro:property name="axle_length" value="0.120"/>
+	<xacro:property name="wheelbase" value="1.800"/>
+	<xacro:property name="hex_hub_dist" value="1.080"/>
+    <xacro:property name="axle_length" value="0.160"/>
 	<xacro:include filename="$(find rbcar_description)/urdf/wheels/suspension_wheel.urdf.xacro" />
 	<!-- Import all available sensors -->
@@ -19,6 +19,6 @@
 	<xacro:property name="PI" value="3.1415926535897931"/>
 	<!-- Wheel parameters -->
-	<xacro:property name="wheel_offset_x" value="1.0" />    <!-- x,y,z in translation from base_link to the center of the wheel -->
-	<xacro:property name="wheel_offset_y" value="0.75" />
+	<xacro:property name="wheel_offset_x" value="0.9" />    <!-- x,y,z in translation from base_link to the center of the wheel -->
+	<xacro:property name="wheel_offset_y" value="0.515" />
 	<xacro:property name="wheel_offset_z" value="0.0" />
 	<!-- Flag to select the high or low quality model -->

File: rbcar_description/urdf/wheels/suspension_wheel.urdf.xacro (robot description, xacro)
@@ -15,7 +15,7 @@
        from a U joint to the corresponding hex hub. wheel_travel is the
        vertical wheel travel. -->
-  <xacro:property name="wheelbase" value="1.650"/>
-  <xacro:property name="hex_hub_dist" value="0.900"/>  <!-- 1.127 0.742 check -->
-  <xacro:property name="axle_length" value="0.120"/>
+  <!-- xacro:property name="wheelbase" value="1.650"/ -->
+  <!-- xacro:property name="hex_hub_dist" value="0.900"/-->  <!-- 1.127 0.742 check -->
+  <!-- xacro:property name="axle_length" value="0.120"/ -->
   <xacro:property name="wheel_travel" value="0.1"/>
   <xacro:property name="shock_z_offset" value="0.05"/>

Commit message: some sensor positions updated

File: rbcar_description/robots/rbcar_ezgo.urdf.xacro (robot description, xacro)
@@ -45,7 +45,7 @@
                     lr_reflect="-1" fr_reflect="-1"/>
 	<!-- SENSORS -->
-    <xacro:sensor_hokuyo3d name="hokuyo3d" parent="base_link">
+    <!-- xacro:sensor_hokuyo3d name="hokuyo3d" parent="base_link">
 		<origin xyz="0.9 0.0 0.450" rpy="0 0.35 0"/>
-	</xacro:sensor_hokuyo3d>
+	</xacro:sensor_hokuyo3d -->
 	<!--xacro:sensor_imu name="imu" parent="base_link">
 		<origin xyz="0.0 0.0 0.170" rpy="0 0 0"/>
@@ -56,11 +56,12 @@
 	</xacro:sensor_imu_hector>
 	<xacro:sensor_gps name="gps" parent="base_link">
-		<origin xyz="-0.25 0 1.25" rpy="0 0 0"/>
+		<origin xyz="0 0 1.55" rpy="0 0 0"/>
 	</xacro:sensor_gps>
 	<xacro:sensor_hokuyo_utm30lx name="hokuyo" parent="base_link">
-		<origin xyz="1.0 0.0 0.33" rpy="0 0 0"/>
+		<origin xyz="1.0 0.0 0.31" rpy="0 0 0"/>
 	</xacro:sensor_hokuyo_utm30lx>
 	<xacro:sensor_hokuyo_urg04lx name="hokuyo1" parent="base_link">
-		<origin xyz="-1.4 0.0 0.33" rpy="0 0 3.1416"/>
+		<!-- origin xyz="0.93 0.0 0.40" rpy="0 0.7854 0"/ -->
+		<origin xyz="0.93 0.0 0.40" rpy="0 0.5236 0"/>
 	</xacro:sensor_hokuyo_urg04lx>
 <!--
