Commit message: modified to work in gazebo

File: rbcar_description/robots/rbcar.urdf (robot description, URDF)
Before this commit: robot rbcar, 12 links, 11 joints
Links:
- added link hokuyo3d_laser_link, mass 1e-5; collision box size=0.1 0.1 0.08; visual mesh filename=package://rbcar_description/meshes/sensors/hokuyo3d.dae
- link left_front_axle_carrier: geometry collision cylinder length=0.1 radius=0.1; visual cylinder length=0.1 radius=0.1
- link left_front_wheel: mass None -> 8.0
- link left_rear_axle_carrier: geometry collision cylinder length=0.1 radius=0.1; visual cylinder length=0.1 radius=0.1
- link left_rear_wheel: mass None -> 8.0
- link left_steering_link: geometry collision cylinder length=0.1 radius=0.1; visual cylinder length=0.1 radius=0.1
- link right_front_axle_carrier: geometry collision cylinder length=0.1 radius=0.1; visual cylinder length=0.1 radius=0.1
- link right_front_wheel: mass None -> 8.0
- link right_rear_axle_carrier: geometry collision cylinder length=0.1 radius=0.1; visual cylinder length=0.1 radius=0.1
- link right_rear_wheel: mass None -> 8.0
- link right_steering_link: geometry collision cylinder length=0.1 radius=0.1; visual cylinder length=0.1 radius=0.1
Joints:
- added joint hokuyo3d_laser_joint: type fixed, parent base_link, child hokuyo3d_laser_link, origin xyz=0.95 0.0 0.1 rpy=0 0 0
- joint left_front_axle: origin rpy=1.57079633 0 0 -> rpy=1.57079633 0 3.14159265
- joint left_front_shock: limit lower=-0.25 upper=0.25 effort=100 velocity=1000 -> lower=-0.05 upper=0.05 effort=100 velocity=1000; origin xyz=0.825                    0.323                    0.25 -> xyz=0.825                    0.33                    0.0; parent chassis -> base_link
- joint left_rear_axle: origin rpy=1.57079633 0 0 -> rpy=1.57079633 0 3.14159265
- joint left_rear_shock: limit lower=-0.25 upper=0.25 effort=100 velocity=1000 -> lower=-0.05 upper=0.05 effort=100 velocity=1000; origin xyz=-0.825                    0.323                    0.25 -> xyz=-0.825                    0.33                    0.0; parent chassis -> base_link
- joint right_front_axle: origin rpy=1.57079633 0 0 -> rpy=1.57079633 0 3.14159265
- joint right_front_shock: limit lower=-0.25 upper=0.25 effort=100 velocity=1000 -> lower=-0.05 upper=0.05 effort=100 velocity=1000; origin xyz=0.825                    -0.323                    0.25 -> xyz=0.825                    -0.33                    0.0; parent chassis -> base_link
- joint right_rear_axle: origin rpy=1.57079633 0 0 -> rpy=1.57079633 0 3.14159265
- joint right_rear_shock: limit lower=-0.25 upper=0.25 effort=100 velocity=1000 -> lower=-0.05 upper=0.05 effort=100 velocity=1000; origin xyz=-0.825                    -0.323                    0.25 -> xyz=-0.825                    -0.33                    0.0; parent chassis -> base_link

File: rbcar_description/robots/rbcar.urdf.xacro (robot description, xacro)
@@ -77,3 +77,6 @@
 	</xacro:sensor_fotonic>
 -->
+  <gazebo>
+    <plugin name="gazebo_ros_control" filename="libgazebo_ros_control.so"/>
+  </gazebo>
 </robot>

File: rbcar_description/urdf/wheels/suspension_wheel.urdf.xacro (robot description, xacro)
@@ -39,4 +39,29 @@
   <xacro:property name="servo_stall_torque" value="50"/>  <!-- check -->
   <xacro:property name="servo_no_load_speed" value="25"/> <!-- check -->
+  <!-- Inertia of a thick-walled cylindrical tube with open ends. Height is
+       measured along the z axis, which is the tube's axis. inner_rad and
+       outer_rad are the tube's inner and outer radii, respectively. -->
+  <xacro:macro name="thick_walled_tube_inertial"
+               params="inner_rad outer_rad height mass">
+    <inertial>
+      <mass value="${mass}"/>
+      <inertia ixx="${(1 / 12) * mass * (3 * (inner_rad * inner_rad +
+                    outer_rad * outer_rad) + height * height)}"
+               ixy="0" ixz="0"
+               iyy="${(1 / 12) * mass * (3 * (inner_rad * inner_rad +
+                    outer_rad * outer_rad) + height * height)}"
+               iyz="0"
+               izz="${mass * (inner_rad * inner_rad +
+                    outer_rad * outer_rad) / 2}"/>
+    </inertial>
+  </xacro:macro>
+  <!-- Null inertial element. This is needed to make the model work with
+       Gazebo. -->
+  <xacro:macro name="null_inertial">
+    <inertial>
+      <mass value="0.001"/>
+      <inertia ixx="0.001" ixy="0" ixz="0" iyy="0.001" iyz="0" izz="0.001"/>
+    </inertial>
+  </xacro:macro>
   <!-- Shock absorber -->
   <xacro:macro name="shock"
@@ -68,4 +93,16 @@
   <xacro:macro name="wheel" params="lr_prefix fr_prefix lr_reflect">
     <link name="${lr_prefix}_${fr_prefix}_axle_carrier">
+	  <!-- visual>
+        <origin xyz="0 0 0"/>
+        <geometry>
+          <cylinder radius="0.1" length="0.1"/>
+        </geometry>
+	  </visual>
+	  <collision>
+        <origin xyz="0 0 0"/>
+        <geometry>
+          <cylinder radius="0.1" length="0.1"/>
+        </geometry>
+	  </collision -->
       <xacro:null_inertial/>
     </link>
@@ -91,4 +128,7 @@
       </actuator>
     </transmission>
+    <gazebo reference="${lr_prefix}_${fr_prefix}_axle_carrier">
+      <material>Gazebo/Black</material>
+    </gazebo>
     <link name="${lr_prefix}_${fr_prefix}_wheel">
       <visual>
@@ -125,4 +165,16 @@
                  child="${lr_prefix}_steering_link"/>
     <link name="${lr_prefix}_steering_link">
+	  <!-- visual>
+		<origin xyz="0 0 0"/>
+        <geometry>
+          <cylinder radius="0.1" length="0.1"/>
+        </geometry>
+	  </visual>
+	  <collision>
+		<origin xyz="0 0 0"/>
+        <geometry>
+          <cylinder radius="0.1" length="0.1"/>
+        </geometry>
+	  </collision -->
       <xacro:null_inertial/>
     </link>
@@ -146,4 +198,7 @@
       </actuator>
     </transmission>
+    <gazebo reference="${lr_prefix}_steering_link">
+      <material>Gazebo/Black</material>
+    </gazebo>
     <xacro:wheel lr_prefix="${lr_prefix}" fr_prefix="${fr_prefix}"
                  lr_reflect="${lr_reflect}"/>

Commit message: updated urdf

File: rbcar_description/robots/rbcar.urdf (robot description, URDF)
Before this commit: robot rbcar, 13 links, 12 joints
Links:
- link base_link: mass 250.0 -> 125.0
- link left_front_axle_carrier: mass None -> 0.001; geometry 
- link left_rear_axle_carrier: mass None -> 0.001; geometry 
- link left_steering_link: mass None -> 0.001; geometry 
- link right_front_axle_carrier: mass None -> 0.001; geometry 
- link right_rear_axle_carrier: mass None -> 0.001; geometry 
- link right_steering_link: mass None -> 0.001; geometry 
Joints:
- joint base_footprint_joint: origin xyz=0 0 0.235 rpy=0 0 0 -> xyz=0 0 0.150 rpy=0 0 0
- joint left_front_axle: limit effort=102.5 velocity=39.02 -> effort=204.95 velocity=39.02
- joint left_rear_axle: limit effort=102.5 velocity=39.02 -> effort=204.95 velocity=39.02
- joint right_front_axle: limit effort=102.5 velocity=39.02 -> effort=204.95 velocity=39.02
- joint right_rear_axle: limit effort=102.5 velocity=39.02 -> effort=204.95 velocity=39.02

Commit message: New controllers

File: rbcar_description/robots/rbcar.urdf (robot description, URDF)
Before this commit: robot rbcar, 13 links, 12 joints
Links:
- removed link hokuyo3d_laser_link
- added link drive_link
- added link front_3d_lidar_base_link, mass 0.564; collision mesh filename=package://robotnik_sensors/meshes/benewake_ce30.stl; visual mesh filename=package://robotnik_sensors/meshes/benewake_ce30.stl
- added link front_3d_lidar_link
- added link gps_base_link, mass 0.001; collision mesh filename=package://robotnik_sensors/meshes/antenna_3GO16.stl scale=1.0 1.0 1.0; visual mesh filename=package://robotnik_sensors/meshes/antenna_3GO16.stl scale=1.0 1.0 1.0
- added link imu_link, mass 0.001; collision box size=.001 .001 .001; visual box size=0.001 0.001 0.001
- added link viper_base_link, mass 0.8; collision box size=0.246 0.035 0.09; visual box size=0.246 0.035 0.09
- added link viper_optical_frame, mass 1E-5
- link base_link: geometry collision mesh filename=package://rbcar_description/meshes/bases/rbcar_chassis.stl; visual mesh filename=package://rbcar_description/meshes/bases/rbcar_chassis.stl
- link left_front_wheel: geometry collision cylinder length=0.322 radius=0.317; visual mesh filename=package://rbcar_description/meshes/wheels/rbcar_wheel.stl
- link left_rear_wheel: geometry collision cylinder length=0.322 radius=0.317; visual mesh filename=package://rbcar_description/meshes/wheels/rbcar_wheel.stl
- link right_front_wheel: geometry collision cylinder length=0.322 radius=0.317; visual mesh filename=package://rbcar_description/meshes/wheels/rbcar_wheel.stl
- link right_rear_wheel: geometry collision cylinder length=0.322 radius=0.317; visual mesh filename=package://rbcar_description/meshes/wheels/rbcar_wheel.stl
Joints:
- removed joint hokuyo3d_laser_joint
- added joint drive_joint: type fixed, parent drive_link, child base_footprint, origin xyz=0.917 0 0 rpy=0 0 0
- added joint front_3d_lidar_base_joint: type fixed, parent base_link, child front_3d_lidar_base_link, origin xyz=1.238 0.0 0.236 rpy=0 0.24396 0
- added joint front_3d_lidar_joint: type fixed, parent front_3d_lidar_base_link, child front_3d_lidar_link
- added joint gps_joint: type fixed, parent base_link, child gps_base_link, origin xyz=-0.17 0 1.5 rpy=0 0 0, axis 0 1 0
- added joint imu_joint: type fixed, parent base_link, child imu_link, origin xyz=0.0 0.0 0.170 rpy=0 0 0, axis 1 0 0
- added joint viper_base_joint: type fixed, parent base_link, child viper_base_link, origin xyz=0.372 0.0 1.354 rpy=0 0.1745 0.0
- added joint viper_optical_joint: type fixed, parent viper_base_link, child viper_optical_frame, origin xyz=0 0 0 rpy=-1.570796 0 -1.570796
- joint base_footprint_joint: origin xyz=0 0 0.150 rpy=0 0 0 -> xyz=0 0 0.317 rpy=0 0 0
- joint left_front_axle: axis 0 0 -1 -> 0 0 1
- joint left_front_shock: origin xyz=0.825                    0.33                    0.0 -> xyz=0.916615                    0.39901                    0.0
- joint left_rear_axle: axis 0 0 -1 -> 0 0 1
- joint left_rear_shock: origin xyz=-0.825                    0.33                    0.0 -> xyz=-0.916615                    0.49925                    0.0
- joint right_front_axle: axis 0 0 -1 -> 0 0 1
- joint right_front_shock: origin xyz=0.825                    -0.33                    0.0 -> xyz=0.916615                    -0.39901                    0.0
- joint right_rear_axle: axis 0 0 -1 -> 0 0 1
- joint right_rear_shock: origin xyz=-0.825                    -0.33                    0.0 -> xyz=-0.916615                    -0.49925                    0.0

File: rbcar_description/robots/rbcar.urdf.xacro (robot description, xacro)
@@ -1,4 +1,5 @@
 <?xml version="1.0"?>
-<robot name="rbcar" xmlns:xacro="http://www.ros.org/wiki/xacro">
+  <robot name="rbcar"
+    xmlns:xacro="http://wiki.ros.org/xacro">
 	<!-- ***************** -->
 	<!-- Imported elements -->
@@ -29,4 +30,5 @@
 	<!-- Gazebo ros control pluggins -->
 	<xacro:ros_control/>
+        <!-- xacro:omni_steering prefix="" publish_tf="true"/-->
 	<!-- Gazebo skid steering pluggins -->
 	<!-- xacro:skid_steering broadcastOdomTF="1"/ -->
@@ -34,23 +36,56 @@
     <!-- Wheels -->
     <xacro:front_wheel lr_prefix="left" fr_prefix="front"
-                       lr_reflect="1" fr_reflect="1"/>
+                       lr_reflect="1" fr_reflect="1" parent="base_link" />
     <xacro:front_wheel lr_prefix="right" fr_prefix="front"
-                       lr_reflect="-1" fr_reflect="1"/>
+                       lr_reflect="-1" fr_reflect="1" parent="base_link" />
     <xacro:rear_wheel lr_prefix="left" fr_prefix="rear"
-                      lr_reflect="1" fr_reflect="-1"/>
+                      lr_reflect="1" fr_reflect="-1" parent="base_link" />
     <xacro:rear_wheel lr_prefix="right" fr_prefix="rear"
-                      lr_reflect="-1" fr_reflect="-1"/>
+                      lr_reflect="-1" fr_reflect="-1" parent="base_link" />
 	<!-- SENSORS -->
     <xacro:sensor_benewake_ce30d prefix="front_3d_lidar" parent="base_link" gpu="true">
-        <origin xyz="1.238 0.0 0.236" rpy="0 0.24396 0"/>
+        <origin xyz="2.155 0.0 0.236" rpy="0 0.24396 0"/>
     </xacro:sensor_benewake_ce30d>
     <xacro:sensor_rubedos_viper prefix="viper" parent="base_link">
-        <origin xyz="0.372 0.0 1.354" rpy="0 0.1745 0.0"/>
+        <origin xyz="1.289 0.0 1.354" rpy="0 0.1745 0.0"/>
     </xacro:sensor_rubedos_viper>
-	<xacro:sensor_imu prefix="imu" parent="base_link">
+	<xacro:sensor_imu_hector prefix="imu" parent="base_link">
 		<origin xyz="0.0 0.0 0.170" rpy="0 0 0"/>
-	</xacro:sensor_imu>
+		<!--<origin xyz="0.917 0.0 0.170" rpy="0 0 0"/>-->
+	</xacro:sensor_imu_hector>
 	<xacro:sensor_gps prefix="gps" parent="base_link">
-		<origin xyz="-0.17 0 1.5" rpy="0 0 0"/>
+		<origin xyz="0.0 0 1.5" rpy="0 0 0"/>
 	</xacro:sensor_gps>
+<gazebo>
+<plugin name="ground_truth_controller" filename="librobotnik_gazebo_ground_truth_odom.so">
+  <alwaysOn>true</alwaysOn>
+  <updateRate>50.0</updateRate>
+  <bodyName>base_link</bodyName>
+  <frameName>base_link_gt</frameName>
+  <worldBodyName>world</worldBodyName>
+  <worldFrameName>world</worldFrameName>
+  <topicName>odom_gt</topicName>
+  <gaussianNoise>0.01</gaussianNoise>
+  <xyzOffset>0.0 0 0</xyzOffset>
+  <rpyOffset>0 0 0</rpyOffset>
+  <applyOffset>False</applyOffset>
+  <broadcastTF>True</broadcastTF>
+</plugin>
+</gazebo>
+<gazebo>
+<plugin name="gps_ground_truth_controller" filename="librobotnik_gazebo_ground_truth_odom.so">
+  <alwaysOn>true</alwaysOn>
+  <updateRate>50.0</updateRate>
+  <bodyName>gps_base_link</bodyName>
+  <frameName>gps_base_link_gt</frameName>
+  <worldBodyName>world</worldBodyName>
+  <worldFrameName>world</worldFrameName>
+  <topicName>odom_gt</topicName>
+  <gaussianNoise>0.01</gaussianNoise>
+  <xyzOffset>0.0 0 0</xyzOffset>
+  <rpyOffset>0 0 0</rpyOffset>
+  <applyOffset>False</applyOffset>
+  <broadcastTF>True</broadcastTF>
+</plugin>
+</gazebo>
 </robot>

File: rbcar_description/urdf/bases/rbcar_base.gazebo.xacro (robot description, xacro)
@@ -1,4 +1,4 @@
 <?xml version="1.0"?>
-<robot xmlns:xacro="http://www.ros.org/wiki/xacro">
+<robot xmlns:xacro="http://wiki.ros.org/xacro">
   <!-- ros control plugin -->
   <xacro:macro name="ros_control">
@@ -12,4 +12,16 @@
 	</xacro:macro>
   <!-- No Ackermann steering plugin -->
+<xacro:macro name="omni_steering" params="prefix publish_tf">
+		<gazebo>
+	    <plugin name="omni_steering" filename="libgazebo_ros_planar_move.so">
+	      <commandTopic>robotnik_base_controller/cmd_vel</commandTopic>
+	      <odometryTopic>robotnik_base_controller/odom</odometryTopic>
+	      <odometryFrame>${prefix}odom</odometryFrame>
+	      <odometryRate>50.0</odometryRate>
+	      <robotBaseFrame>${prefix}base_footprint</robotBaseFrame>
+	      <publishTF>${publish_tf}</publishTF>
+	    </plugin>
+	  </gazebo>
+  </xacro:macro>
   <gazebo reference="base_footprint">
     <material>Gazebo/Green</material>

File: rbcar_description/urdf/bases/rbcar_base.urdf.xacro (robot description, xacro)
@@ -1,4 +1,4 @@
 <?xml version="1.0"?>
-<robot name="rbcar" xmlns:xacro="http://www.ros.org/wiki/xacro">
+<robot name="rbcar" xmlns:xacro="http://wiki.ros.org/xacro">
   <xacro:include filename="$(find rbcar_description)/urdf/bases/rbcar_base.gazebo.xacro" />
   <xacro:macro name="rbcar_base" params="name publish_bf hq">
@@ -35,17 +35,17 @@
     <inertial>
       <mass value="125.0" />
-      <origin xyz="0 0 0" />
+      <origin xyz="0.917 0 0" />
       <inertia  ixx="1.391" ixy="0.004"  ixz="0.0"  iyy="6.853"  iyz="0.0"  izz="6.125" />
     </inertial>
     <visual>
-       <origin xyz="0 0 0" rpy="0 0 0" />
+       <origin xyz="0.917 0 0" rpy="0 0 0" />
        <xacro:if value="${hq}">
        <geometry>
-	     <mesh filename="package://rbcar_description/meshes/bases/rbcar_chassis.STL"/>
+	     <mesh filename="package://rbcar_description/meshes/bases/rbcar_chassis.stl"/>
        </geometry>
        </xacro:if>
        <xacro:unless value="${hq}">
        <geometry>
-	     <mesh filename="package://rbcar_description/meshes/bases/rbcar_chassis.STL"/>
+	     <mesh filename="package://rbcar_description/meshes/bases/rbcar_chassis.stl"/>
        </geometry>
        </xacro:unless>
@@ -55,7 +55,7 @@
     </visual>
     <collision>
-       <origin xyz="0 0 0" rpy="0 0 0 " />
+       <origin xyz="0.917 0 0" rpy="0 0 0 " />
        <geometry>
-         <mesh filename="package://rbcar_description/meshes/bases/rbcar_chassis.STL"/>
+         <mesh filename="package://rbcar_description/meshes/bases/rbcar_chassis.stl"/>
        </geometry>
     </collision>

File: rbcar_description/urdf/wheels/suspension_wheel.urdf.xacro (robot description, xacro)
@@ -1,4 +1,4 @@
 <?xml version="1.0"?>
-<robot name="wheel" xmlns:xacro="http://www.ros.org/wiki/xacro">
+<robot name="wheel" xmlns:xacro="http://wiki.ros.org/xacro">
   <!-- hub_dia and tire_dia are the diameters of the hub and tire,
        respectively. hex_hub_depth is the distance that the hex hub is

File: rbcar_description/urdf/wheels/suspension_wheel_v2.urdf.xacro (robot description, xacro)
@@ -1,4 +1,4 @@
 <?xml version="1.0"?>
-<robot name="wheel" xmlns:xacro="http://www.ros.org/wiki/xacro">
+<robot name="wheel" xmlns:xacro="http://wiki.ros.org/xacro">
   <!-- hub_dia and tire_dia are the diameters of the hub and tire,
        respectively. hex_hub_depth is the distance that the hex hub is
@@ -71,7 +71,7 @@
   <!-- Shock absorber -->
   <xacro:macro name="shock"
-               params="lr_prefix fr_prefix lr_reflect fr_reflect child">
+               params="lr_prefix fr_prefix lr_reflect fr_reflect child parent">
     <joint name="${lr_prefix}_${fr_prefix}_shock" type="prismatic">
-      <parent link="base_link"/>
+      <parent link="${parent}"/>
       <child link="${child}"/>
       <xacro:if value="${fr_prefix=='front'}">
@@ -81,5 +81,5 @@
         <xacro:property name="hex_hub_dist" value="1.2385"/>
       </xacro:if>
-      <origin xyz="${fr_reflect * wheelbase / 2}
+      <origin xyz="${fr_reflect * wheelbase / 2 + 0.917}
                    ${lr_reflect * ((hex_hub_dist / 2) - axle_length)}
                    ${(wheel_travel / 2) - shock_z_offset}"/>
@@ -153,5 +153,5 @@
         <geometry>
           <!--cylinder radius="${tire_dia / 2}" length="${tire_width}"/-->
-          <mesh filename="package://rbcar_description/meshes/wheels/rbcar_wheel.STL"/>
+          <mesh filename="package://rbcar_description/meshes/wheels/rbcar_wheel.stl"/>
         </geometry>
         <material name="tire_mat"/>
@@ -176,8 +176,8 @@
   <!-- Front wheel -->
   <xacro:macro name="front_wheel"
-               params="lr_prefix fr_prefix lr_reflect fr_reflect">
+               params="lr_prefix fr_prefix lr_reflect fr_reflect parent">
     <xacro:shock lr_prefix="${lr_prefix}" fr_prefix="${fr_prefix}"
                  lr_reflect="${lr_reflect}" fr_reflect="${fr_reflect}"
-                 child="${lr_prefix}_steering_link"/>
+                 child="${lr_prefix}_steering_link" parent="${parent}"/>
     <link name="${lr_prefix}_steering_link">
 	  <!-- visual>
@@ -220,8 +220,8 @@
   <!-- Rear wheel -->
   <xacro:macro name="rear_wheel"
-               params="lr_prefix fr_prefix lr_reflect fr_reflect">
+               params="lr_prefix fr_prefix lr_reflect fr_reflect parent">
     <xacro:shock lr_prefix="${lr_prefix}" fr_prefix="${fr_prefix}"
                  lr_reflect="${lr_reflect}" fr_reflect="${fr_reflect}"
-                 child="${lr_prefix}_${fr_prefix}_axle_carrier"/>
+                 child="${lr_prefix}_${fr_prefix}_axle_carrier" parent="${parent}"/>
     <xacro:wheel lr_prefix="${lr_prefix}" fr_prefix="${fr_prefix}"
                  lr_reflect="${lr_reflect}"/>
