Commit message: new branch to melex

File: rbcar_description/robots/rbcar.urdf (robot description, URDF)
Before this commit: robot rbcar, 19 links, 18 joints
Links:
- removed link drive_link
- removed link front_3d_lidar_base_link
- removed link front_3d_lidar_link
- removed link gps_base_link
- removed link imu_link
- removed link viper_base_link
- removed link viper_optical_frame
- added link hokuyo3d_laser_link, mass 1e-5; collision box size=0.1 0.1 0.08; visual mesh filename=package://rbcar_description/meshes/sensors/hokuyo3d.dae
- link base_link: geometry collision mesh filename=package://rbcar_description/meshes/bases/rbcar_chassis.dae; visual mesh filename=package://rbcar_description/meshes/bases/rbcar_chassis.dae
- link left_front_wheel: geometry collision cylinder length=0.2 radius=0.235; visual cylinder length=0.2 radius=0.235
- link left_rear_wheel: geometry collision cylinder length=0.2 radius=0.235; visual cylinder length=0.2 radius=0.235
- link right_front_wheel: geometry collision cylinder length=0.2 radius=0.235; visual cylinder length=0.2 radius=0.235
- link right_rear_wheel: geometry collision cylinder length=0.2 radius=0.235; visual cylinder length=0.2 radius=0.235
Joints:
- removed joint drive_joint
- removed joint front_3d_lidar_base_joint
- removed joint front_3d_lidar_joint
- removed joint gps_joint
- removed joint imu_joint
- removed joint viper_base_joint
- removed joint viper_optical_joint
- added joint hokuyo3d_laser_joint: type fixed, parent base_link, child hokuyo3d_laser_link, origin xyz=0.95 0.0 0.1 rpy=0 0 0
- joint base_footprint_joint: origin xyz=0 0 0.317 rpy=0 0 0 -> xyz=0 0 0.150 rpy=0 0 0
- joint left_front_axle: axis 0 0 1 -> 0 0 -1
- joint left_front_shock: origin xyz=0.916615                    0.39901                    0.0 -> xyz=0.825                    0.33                    0.0
- joint left_rear_axle: axis 0 0 1 -> 0 0 -1
- joint left_rear_shock: origin xyz=-0.916615                    0.49925                    0.0 -> xyz=-0.825                    0.33                    0.0
- joint right_front_axle: axis 0 0 1 -> 0 0 -1
- joint right_front_shock: origin xyz=0.916615                    -0.39901                    0.0 -> xyz=0.825                    -0.33                    0.0
- joint right_rear_axle: axis 0 0 1 -> 0 0 -1
- joint right_rear_shock: origin xyz=-0.916615                    -0.49925                    0.0 -> xyz=-0.825                    -0.33                    0.0

File: rbcar_description/robots/rbcar_.urdf.xacro (robot description, xacro)
@@ -6,7 +6,7 @@
 	<!-- First we import all posible elements defined in the urdf.xacro files. All these elements are defined as macro:xacros -->
 	<!-- Import Robotnik CAR base elements -->
-	<xacro:include filename="$(find rbcar_description)/urdf/bases/rbcar_base_v2.urdf.xacro" />
+	<xacro:include filename="$(find rbcar_description)/urdf/bases/rbcar_base.urdf.xacro" />
 	<!-- Import Robotnik CAR wheels -->
-	<xacro:include filename="$(find rbcar_description)/urdf/wheels/suspension_wheel_v2.urdf.xacro" />
+	<xacro:include filename="$(find rbcar_description)/urdf/wheels/suspension_wheel.urdf.xacro" />
 	<!-- Import all available sensors -->
 	<xacro:include filename="$(find robotnik_sensors)/urdf/all_sensors.urdf.xacro" />
@@ -16,6 +16,6 @@
 	<xacro:property name="PI" value="3.1415926535897931"/>
 	<!-- Wheel parameters -->
-	<xacro:property name="wheel_offset_x" value="1.0" />    <!-- x,y,z in translation from base_link to the center of the wheel -->
-	<xacro:property name="wheel_offset_y" value="0.75" />
+	<xacro:property name="wheel_offset_x" value="1.25" />    <!-- x,y,z in translation from base_link to the center of the wheel -->
+	<xacro:property name="wheel_offset_y" value="0.525" />
 	<xacro:property name="wheel_offset_z" value="0.0" />
 	<!-- Flag to select the high or low quality model -->
@@ -34,11 +34,11 @@
   <!-- Wheels -->
   <xacro:front_wheel lr_prefix="left" fr_prefix="front"
-                     lr_reflect="1" fr_reflect="1" parent="base_link" />
+                     lr_reflect="1" fr_reflect="1"/>
   <xacro:front_wheel lr_prefix="right" fr_prefix="front"
-                     lr_reflect="-1" fr_reflect="1" parent="base_link" />
+                     lr_reflect="-1" fr_reflect="1"/>
   <xacro:rear_wheel lr_prefix="left" fr_prefix="rear"
-                    lr_reflect="1" fr_reflect="-1" parent="base_link" />
+                    lr_reflect="1" fr_reflect="-1"/>
   <xacro:rear_wheel lr_prefix="right" fr_prefix="rear"
-                    lr_reflect="-1" fr_reflect="-1" parent="base_link" />
+                    lr_reflect="-1" fr_reflect="-1"/>
 	<!-- SENSORS -->
     <xacro:sensor_sick_s3000 prefix="front_laser" parent="base_link">
@@ -77,41 +77,7 @@
 	</xacro:sensor_fotonic>
 -->
-    <xacro:elevator parent="base_link">
-		<origin xyz="0.0 0.0 0.6" rpy="0 0 0"/>
-	</xacro:elevator>
-    <xacro:sensor_axis prefix="front_ptz_camera" parent="elevator_link" far="300" near="0.08">
-            <origin xyz="0 0 0" rpy="0 0 0"/>
-    </xacro:sensor_axis>
-<gazebo>
-<plugin name="ground_truth_controller" filename="librobotnik_gazebo_ground_truth_odom.so">
-  <alwaysOn>true</alwaysOn>
-  <updateRate>50.0</updateRate>
-  <bodyName>base_link</bodyName>
-  <frameName>base_link_gt</frameName>
-  <worldBodyName>world</worldBodyName>
-  <worldFrameName>world</worldFrameName>
-  <topicName>odom_gt</topicName>
-  <gaussianNoise>0.01</gaussianNoise>
-  <xyzOffset>0.0 0 0</xyzOffset>
-  <rpyOffset>0 0 0</rpyOffset>
-  <applyOffset>False</applyOffset>
-  <broadcastTF>True</broadcastTF>
-</plugin>
-</gazebo>
-<gazebo>
-<plugin name="gps_ground_truth_controller" filename="librobotnik_gazebo_ground_truth_odom.so">
-  <alwaysOn>true</alwaysOn>
-  <updateRate>50.0</updateRate>
-  <bodyName>gps_base_link</bodyName>
-  <frameName>gps_base_link_gt</frameName>
-  <worldBodyName>world</worldBodyName>
-  <worldFrameName>world</worldFrameName>
-  <topicName>odom_gt</topicName>
-  <gaussianNoise>0.01</gaussianNoise>
-  <xyzOffset>0.0 0 0</xyzOffset>
-  <rpyOffset>0 0 0</rpyOffset>
-  <applyOffset>False</applyOffset>
-  <broadcastTF>True</broadcastTF>
-</plugin>
-</gazebo>
+  <!-- gazebo>
+    <plugin name="gazebo_ros_control" filename="libgazebo_ros_control.so"/>
+  </gazebo -->
+  <!-- ros control plugin -->
 </robot>

File: rbcar_description/urdf/bases/rbcar_base_v2.urdf.xacro (robot description, xacro)
@@ -42,13 +42,13 @@
        <xacro:if value="${hq}">
        <geometry>
-	     <mesh filename="package://rbcar_description/meshes/bases/rbcar_chassis.dae"/>
+	     <mesh filename="package://rbcar_description/meshes/bases/rbcar_chassis_v2.STL"/>
        </geometry>
        </xacro:if>
        <xacro:unless value="${hq}">
        <geometry>
-	     <mesh filename="package://rbcar_description/meshes/bases/rbcar_chassis.dae"/>
+	     <mesh filename="package://rbcar_description/meshes/bases/rbcar_chassis_v2.STL"/>
        </geometry>
        </xacro:unless>
-       <material name="darkgrey">
+       <material name="white">
          <color rgba="0.1 0.1 0.1 1"/>
        </material>
@@ -57,5 +57,5 @@
        <origin xyz="0 0 0" rpy="0 0 0 " />
        <geometry>
-         <mesh filename="package://rbcar_description/meshes/bases/rbcar_chassis.dae"/>
+         <mesh filename="package://rbcar_description/meshes/bases/rbcar_chassis_v2.STL"/>
        </geometry>
     </collision>

File: rbcar_description/urdf/wheels/suspension_wheel.urdf.xacro (robot description, xacro)
@@ -1,4 +1,4 @@
 <?xml version="1.0"?>
-<robot name="wheel" xmlns:xacro="http://wiki.ros.org/xacro">
+<robot name="wheel" xmlns:xacro="http://www.ros.org/wiki/xacro">
   <!-- hub_dia and tire_dia are the diameters of the hub and tire,
        respectively. hex_hub_depth is the distance that the hex hub is

File: rbcar_description/urdf/wheels/suspension_wheel_v2.urdf.xacro (robot description, xacro)
@@ -7,6 +7,6 @@
        axle_length. -->
   <xacro:property name="hub_dia" value="0.235"/>
-  <xacro:property name="tire_dia" value="0.634"/>
-  <xacro:property name="tire_width" value="0.322"/>
+  <xacro:property name="tire_dia" value="0.440"/>
+  <xacro:property name="tire_width" value="0.195"/>
   <xacro:property name="hex_hub_depth" value="0.120"/> <!-- or +0.072 -->
   <xacro:property name="wheel_mass" value="8.0"/>   <!-- check -->
@@ -15,6 +15,6 @@
        from a U joint to the corresponding hex hub. wheel_travel is the
        vertical wheel travel. -->
-  <xacro:property name="wheelbase" value="1.83323"/>
-  <!--xacro:property name="hex_hub_dist" value="1.2385"/-->  <!-- 1.127 0.742 0.900 check -->
+  <xacro:property name="wheelbase" value="2.5"/>
+  <xacro:property name="hex_hub_dist" value="0.9191"/>  <!-- 1.127 0.742 0.900 check -->
   <xacro:property name="axle_length" value="0.120"/>
   <xacro:property name="wheel_travel" value="0.1"/>
@@ -153,6 +153,5 @@
         </xacro:if>
         <geometry>
-          <!--cylinder radius="${tire_dia / 2}" length="${tire_width}"/-->
-          <mesh filename="package://rbcar_description/meshes/wheels/rbcar_wheel.stl"/>
+          <cylinder radius="${tire_dia / 2}" length="${tire_width}"/>
         </geometry>
         <material name="tire_mat"/>
