Commit message: changed 3d laser pos

File: rbcar_description/robots/rbcar.urdf.xacro (robot description, xacro)
@@ -43,5 +43,5 @@
 	<!-- SENSORS -->
     <xacro:sensor_hokuyo3d name="hokuyo3d" parent="base_link">
-		<origin xyz="1.0 0.0 0.1" rpy="0 0 0"/>
+		<origin xyz="0.95 0.0 0.1" rpy="0 0 0"/>
 	</xacro:sensor_hokuyo3d>
 	<!--xacro:sensor_hokuyo_utm30lx name="hokuyo" parent="base_link">

Commit message: updated model - 1st working in gazebo

File: rbcar_description/robots/rbcar.urdf.xacro (robot description, xacro)
@@ -77,6 +77,7 @@
 	</xacro:sensor_fotonic>
 -->
-  <gazebo>
+  <!-- gazebo>
     <plugin name="gazebo_ros_control" filename="libgazebo_ros_control.so"/>
-  </gazebo>
+  </gazebo -->
+  <!-- ros control plugin -->
 </robot>

File: rbcar_description/urdf/bases/rbcar_base.gazebo.xacro (robot description, xacro)
@@ -2,8 +2,8 @@
 <robot xmlns:xacro="http://ros.org/wiki/xacro">
   <!-- ros control plugin -->
-  <!-- xacro:macro name="ros_control">
+  <xacro:macro name="ros_control">
     <gazebo>
       <plugin name="ros_control" filename="libgazebo_ros_control.so">
-        <robotNamespace>/summit_xl</robotNamespace>
+        <robotNamespace>/rbcar</robotNamespace>
         <robotParam>robot_description</robotParam>
         <controlPeriod>0.003</controlPeriod>
@@ -11,38 +11,6 @@
       </plugin>
     </gazebo>
-	</xacro:macro -->
-	<!-- skid steering plugin -->
-	<xacro:macro name="skid_steering" params="broadcastOdomTF">
-    <gazebo>
-      <plugin name="skid_steer_drive_controller" filename="libgazebo_ros_skid_steer_drive.so">
-				<robotNamespace>/summit_xl</robotNamespace>
-		    <updateRate>100.0</updateRate>
-		    <leftFrontJoint>joint_front_left_wheel</leftFrontJoint>
-		    <rightFrontJoint>joint_front_right_wheel</rightFrontJoint>
-		    <leftRearJoint>joint_back_left_wheel</leftRearJoint>
-		    <rightRearJoint>joint_back_right_wheel</rightRearJoint>
-		    <wheelSeparation>0.468</wheelSeparation>
-		    <wheelDiameter>0.234</wheelDiameter>
-		    <robotBaseFrame>base_footprint</robotBaseFrame>
-		    <torque>25</torque>
-		    <topicName>cmd_vel</topicName>
-		    <commandTopic>robot_control/command</commandTopic>
-		    <odometryTopic>odom</odometryTopic>
-		    <odometryFrame>/odom</odometryFrame>
-		    <broadcastTF>${broadcastOdomTF}</broadcastTF>
-      </plugin>
-    </gazebo>
-  </xacro:macro>
-  <xacro:macro name="omni_steering">
-		<gazebo>
-	    <plugin name="omni_steering" filename="libgazebo_ros_planar_move.so">
-	      <commandTopic>/summit_xl/robot_control/command</commandTopic>
-	      <odometryTopic>/summit_xl/odom</odometryTopic>
-	      <odometryFrame>odom</odometryFrame>
-	      <odometryRate>20.0</odometryRate>
-	      <robotBaseFrame>base_footprint</robotBaseFrame>
-	    </plugin>
-	  </gazebo>
-  </xacro:macro>
+	</xacro:macro>
+  <!-- No Ackermann steering plugin -->
   <gazebo reference="base_footprint">
     <material>Gazebo/Green</material>

File: rbcar_description/urdf/bases/rbcar_base.urdf.xacro (robot description, xacro)
@@ -34,5 +34,5 @@
   <link name="base_link">
     <inertial>
-      <mass value="250.0" />
+      <mass value="125.0" />
       <origin xyz="0 0 0" />
       <inertia  ixx="1.391" ixy="0.004"  ixz="0.0"  iyy="6.853"  iyz="0.0"  izz="6.125" />

Commit message: added imu, needed for odometry estimation

File: rbcar_description/robots/rbcar.urdf.xacro (robot description, xacro)
@@ -45,4 +45,7 @@
 		<origin xyz="0.95 0.0 0.1" rpy="0 0 0"/>
 	</xacro:sensor_hokuyo3d>
+	<xacro:sensor_imu name="imu" parent="base_link">
+		<origin xyz="0.0 0.0 0.170" rpy="0 0 0"/>
+	</xacro:sensor_imu>
 	<!--xacro:sensor_hokuyo_utm30lx name="hokuyo" parent="base_link">
 		<origin xyz="0.0 0.0 0.33" rpy="0 0 0"/>
@@ -56,7 +59,4 @@
 		<origin xyz="0.19 0 0.17" rpy="0 ${15*PI/180} 0"/>
 	</xacro:sensor_axis>
-	<xacro:sensor_imu name="imu" parent="base_link">
-		<origin xyz="-0.18 0.0 0.170" rpy="0 0 0"/>
-	</xacro:sensor_imu>
 	<xacro:sensor_gps name="gps" parent="base_link">
 		<origin xyz="-0.22 0 0.275" rpy="0 0 0"/>

Commit message: rbcar_description: changing 3d sensor position to fit with the real model

File: rbcar_description/robots/rbcar.urdf.xacro (robot description, xacro)
@@ -43,5 +43,5 @@
 	<!-- SENSORS -->
     <xacro:sensor_hokuyo3d name="hokuyo3d" parent="base_link">
-		<origin xyz="0.95 0.0 0.1" rpy="0 0 0"/>
+		<origin xyz="0.9 0.0 0.450" rpy="0 0.35 0"/>
 	</xacro:sensor_hokuyo3d>
 	<xacro:sensor_imu name="imu" parent="base_link">

File: rbcar_description/urdf/bases/rbcar_base.urdf.xacro (robot description, xacro)
@@ -25,5 +25,5 @@
     </link>
     <joint name="base_footprint_joint" type="fixed">
-      <origin xyz="0 0 0.150" rpy="0 0 0" />  <!-- height is the clearance -->
+      <origin xyz="0 0 0.235" rpy="0 0 0" />  <!-- height is the clearance -->
       <parent link="base_footprint"/>
       <child link="base_link" />

Commit message: added gps and hector imu to description

File: rbcar_description/robots/rbcar.urdf.xacro (robot description, xacro)
@@ -45,7 +45,14 @@
 		<origin xyz="0.9 0.0 0.450" rpy="0 0.35 0"/>
 	</xacro:sensor_hokuyo3d>
-	<xacro:sensor_imu name="imu" parent="base_link">
+	<!--xacro:sensor_imu name="imu" parent="base_link">
 		<origin xyz="0.0 0.0 0.170" rpy="0 0 0"/>
-	</xacro:sensor_imu>
+	</xacro:sensor_imu -->
+	<!-- Imu with hector plugin -->
+	<xacro:sensor_imu_hector name="imu" parent="base_link">
+		<origin xyz="0.0 0.0 0.0" rpy="0 0 0"/>
+	</xacro:sensor_imu_hector>
+	<xacro:sensor_gps name="gps" parent="base_link">
+		<origin xyz="-0.25 0 1.25" rpy="0 0 0"/>
+	</xacro:sensor_gps>
 	<!--xacro:sensor_hokuyo_utm30lx name="hokuyo" parent="base_link">
 		<origin xyz="0.0 0.0 0.33" rpy="0 0 0"/>
@@ -56,10 +63,9 @@
 	</xacro:sensor_hokuyo_urg04lx>
 -->
-	<!-- xacro:sensor_axis name="camera" parent="base_link">
+<!--
+	<xacro:sensor_axis name="camera" parent="base_link">
 		<origin xyz="0.19 0 0.17" rpy="0 ${15*PI/180} 0"/>
 	</xacro:sensor_axis>
-	<xacro:sensor_gps name="gps" parent="base_link">
-		<origin xyz="-0.22 0 0.275" rpy="0 0 0"/>
-	</xacro:sensor_gps -->
+-->
 <!--
 	<xacro:sensor_asus_xtion_pro name="xtion_pro" parent="base_link">

Commit message: added laser sensors to robot

File: rbcar_description/robots/rbcar.urdf.xacro (robot description, xacro)
@@ -55,12 +55,10 @@
 		<origin xyz="-0.25 0 1.25" rpy="0 0 0"/>
 	</xacro:sensor_gps>
-	<!--xacro:sensor_hokuyo_utm30lx name="hokuyo" parent="base_link">
-		<origin xyz="0.0 0.0 0.33" rpy="0 0 0"/>
-	</xacro:sensor_hokuyo_utm30lx -->
-<!--
+	<xacro:sensor_hokuyo_utm30lx name="hokuyo" parent="base_link">
+		<origin xyz="1.0 0.0 0.33" rpy="0 0 0"/>
+	</xacro:sensor_hokuyo_utm30lx>
 	<xacro:sensor_hokuyo_urg04lx name="hokuyo1" parent="base_link">
-		<origin xyz="-0.1 0.0 0.33" rpy="0 0 0"/>
+		<origin xyz="-1.4 0.0 0.33" rpy="0 0 3.1416"/>
 	</xacro:sensor_hokuyo_urg04lx>
--->
 <!--
 	<xacro:sensor_axis name="camera" parent="base_link">

Commit message: description: modifying position of the wheels

File: rbcar_description/robots/rbcar.urdf.xacro (robot description, xacro)
@@ -8,7 +8,4 @@
 	<xacro:include filename="$(find rbcar_description)/urdf/bases/rbcar_base.urdf.xacro" />
 	<!-- Import Robotnik CAR wheels -->
-    <xacro:property name="wheelbase" value="1.650"/>
-    <xacro:property name="hex_hub_dist" value="0.900"/>
-    <xacro:property name="axle_length" value="0.120"/>
 	<xacro:include filename="$(find rbcar_description)/urdf/wheels/suspension_wheel.urdf.xacro" />
 	<!-- Import all available sensors -->

File: rbcar_description/urdf/bases/rbcar_base.urdf.xacro (robot description, xacro)
@@ -6,4 +6,5 @@
   <xacro:property name="PI" value="3.1415926535897931"/>
   <xacro:property name="wheel_width" value="0.175" />
+  <xacro:property name="clearance" value="0.235" />
   <!-- BASE FOOTPRINT -->
   <xacro:if value="${publish_bf}">

File: rbcar_description/urdf/wheels/suspension_wheel.urdf.xacro (robot description, xacro)
@@ -15,7 +15,7 @@
        from a U joint to the corresponding hex hub. wheel_travel is the
        vertical wheel travel. -->
-  <!-- xacro:property name="wheelbase" value="1.650"/ -->
-  <!-- xacro:property name="hex_hub_dist" value="0.900"/-->  <!-- 1.127 0.742 check -->
-  <!-- xacro:property name="axle_length" value="0.120"/ -->
+  <xacro:property name="wheelbase" value="1.650"/>
+  <xacro:property name="hex_hub_dist" value="0.900"/>  <!-- 1.127 0.742 0.900 check -->
+  <xacro:property name="axle_length" value="0.120"/>
   <xacro:property name="wheel_travel" value="0.1"/>
   <xacro:property name="shock_z_offset" value="0.05"/>
@@ -77,5 +77,6 @@
       <origin xyz="${fr_reflect * wheelbase / 2}
                    ${lr_reflect * ((hex_hub_dist / 2) - axle_length)}
-                   ${(wheel_travel / 2) - shock_z_offset}"/>
+                   ${-wheel_travel}"/>
+                  <!-- ${(wheel_travel / 2) - shock_z_offset}"/-->
       <axis xyz="0 0 -1"/>
       <limit lower="${-wheel_travel / 2}" upper="${wheel_travel / 2}"
@@ -86,5 +87,5 @@
       <type>transmission_interface/SimpleTransmission</type>
       <joint name="${lr_prefix}_${fr_prefix}_shock">
-        <hardwareInterface>EffortJointInterface</hardwareInterface>
+        <hardwareInterface>hardware_interface/EffortJointInterface</hardwareInterface>
       </joint>
       <actuator name="${lr_prefix}_${fr_prefix}_shock_act">
@@ -123,6 +124,6 @@
       <type>transmission_interface/SimpleTransmission</type>
       <joint name="${lr_prefix}_${fr_prefix}_axle">
-        <!-- hardwareInterface>EffortJointInterface</hardwareInterface -->
-        <hardwareInterface>VelocityJointInterface</hardwareInterface>
+        <!-- hardwareInterface>hardware_interface/EffortJointInterface</hardwareInterface -->
+        <hardwareInterface>hardware_interface/VelocityJointInterface</hardwareInterface>
       </joint>
       <actuator name="${lr_prefix}_${fr_prefix}_axle_act">
@@ -191,5 +192,5 @@
       <type>transmission_interface/SimpleTransmission</type>
       <joint name="${lr_prefix}_steering_joint">
-        <hardwareInterface>EffortJointInterface</hardwareInterface>
+        <hardwareInterface>hardware_interface/EffortJointInterface</hardwareInterface>
       </joint>
       <actuator name="${lr_prefix}_steering_act">

Commit message: cleaned rbcar description

File: rbcar_description/robots/rbcar.urdf.xacro (robot description, xacro)
@@ -2,90 +2,58 @@
   <robot name="rbcar"
     xmlns:xacro="http://wiki.ros.org/xacro">
-	<!-- ***************** -->
-	<!-- Imported elements -->
-	<!-- ***************** -->
-	<!-- First we import all posible elements defined in the urdf.xacro files. All these elements are defined as macro:xacros -->
-	<!-- Import Robotnik CAR base elements -->
-	<xacro:include filename="$(find rbcar_description)/urdf/bases/rbcar_base.urdf.xacro" />
-	<!-- Import Robotnik CAR wheels -->
-	<xacro:include filename="$(find rbcar_description)/urdf/wheels/suspension_wheel_v2.urdf.xacro" />
-	<!-- Import all available sensors -->
-	<xacro:include filename="$(find robotnik_sensors)/urdf/all_sensors.urdf.xacro" />
-	<!-- ***************** -->
-	<!-- Global parameters -->
-	<!-- ***************** -->
-	<xacro:property name="PI" value="3.1415926535897931"/>
-	<!-- Wheel parameters -->
-	<xacro:property name="wheel_offset_x" value="1.0" />    <!-- x,y,z in translation from base_link to the center of the wheel -->
-	<xacro:property name="wheel_offset_y" value="0.75" />
-	<xacro:property name="wheel_offset_z" value="0.0" />
-	<!-- Flag to select the high or low quality model -->
-	<xacro:property name="hq" value="true" />
-	<!-- *************** -->
-	<!-- Robots Elements -->
-	<!-- *************** -->
-	<!-- Here we create the robot elements using the xacro:macros imported at the beggining of this file -->
-	<!-- Summit XL base -->
-	<xacro:rbcar_base name="rbcar" publish_bf="true" hq="${hq}" />
-	<!-- Gazebo ros control pluggins -->
-	<xacro:ros_control/>
+  <!-- ***************** -->
+  <!-- Imported elements -->
+  <!-- ***************** -->
+  <!-- First we import all posible elements defined in the urdf.xacro files. All these elements are defined as macro:xacros -->
+  <!-- Import Robotnik CAR base elements -->
+  <xacro:include filename="$(find rbcar_description)/urdf/bases/rbcar_base.urdf.xacro" />
+  <!-- Import Robotnik CAR wheels -->
+  <xacro:include filename="$(find rbcar_description)/urdf/wheels/suspension_wheel_v2.urdf.xacro" />
+  <!-- Import all available sensors -->
+  <xacro:include filename="$(find robotnik_sensors)/urdf/all_sensors.urdf.xacro" />
+  <!-- ***************** -->
+  <!-- Global parameters -->
+  <!-- ***************** -->
+  <xacro:property name="PI" value="3.1415926535897931"/>
+  <!-- Wheel parameters -->
+  <xacro:property name="wheel_offset_x" value="1.0" />    <!-- x,y,z in translation from base_link to the center of the wheel -->
+  <xacro:property name="wheel_offset_y" value="0.75" />
+  <xacro:property name="wheel_offset_z" value="0.0" />
+  <!-- Flag to select the high or low quality model -->
+  <xacro:property name="hq" value="true" />
+  <!-- *************** -->
+  <!-- Robots Elements -->
+  <!-- *************** -->
+  <!-- Here we create the robot elements using the xacro:macros imported at the beggining of this file -->
+  <!-- Summit XL base -->
+  <xacro:rbcar_base name="rbcar" publish_bf="true" hq="${hq}" />
+  <!-- Gazebo ros control pluggins -->
+  <xacro:ros_control/>
         <!-- xacro:omni_steering prefix="" publish_tf="true"/-->
-	<!-- Gazebo skid steering pluggins -->
-	<!-- xacro:skid_steering broadcastOdomTF="1"/ -->
-	<!-- WHEELS -->
-    <!-- Wheels -->
-    <xacro:front_wheel lr_prefix="left" fr_prefix="front"
-                       lr_reflect="1" fr_reflect="1" parent="base_link" />
-    <xacro:front_wheel lr_prefix="right" fr_prefix="front"
-                       lr_reflect="-1" fr_reflect="1" parent="base_link" />
-    <xacro:rear_wheel lr_prefix="left" fr_prefix="rear"
-                      lr_reflect="1" fr_reflect="-1" parent="base_link" />
-    <xacro:rear_wheel lr_prefix="right" fr_prefix="rear"
-                      lr_reflect="-1" fr_reflect="-1" parent="base_link" />
-	<!-- SENSORS -->
-    <xacro:sensor_benewake_ce30d prefix="front_3d_lidar" parent="base_link" gpu="true">
-        <origin xyz="2.155 0.0 0.236" rpy="0 0.24396 0"/>
-    </xacro:sensor_benewake_ce30d>
-    <xacro:sensor_rubedos_viper prefix="viper" parent="base_link">
-        <origin xyz="1.289 0.0 1.354" rpy="0 0.1745 0.0"/>
-    </xacro:sensor_rubedos_viper>
-	<xacro:sensor_imu_hector prefix="imu" parent="base_link">
-		<origin xyz="0.0 0.0 0.170" rpy="0 0 0"/>
-		<!--<origin xyz="0.917 0.0 0.170" rpy="0 0 0"/>-->
-	</xacro:sensor_imu_hector>
-	<xacro:sensor_gps prefix="gps" parent="base_link">
-		<origin xyz="0.0 0 1.5" rpy="0 0 0"/>
-	</xacro:sensor_gps>
-<gazebo>
-<plugin name="ground_truth_controller" filename="librobotnik_gazebo_ground_truth_odom.so">
-  <alwaysOn>true</alwaysOn>
-  <updateRate>50.0</updateRate>
-  <bodyName>base_link</bodyName>
-  <frameName>base_link_gt</frameName>
-  <worldBodyName>world</worldBodyName>
-  <worldFrameName>world</worldFrameName>
-  <topicName>odom_gt</topicName>
-  <gaussianNoise>0.01</gaussianNoise>
-  <xyzOffset>0.0 0 0</xyzOffset>
-  <rpyOffset>0 0 0</rpyOffset>
-  <applyOffset>False</applyOffset>
-  <broadcastTF>True</broadcastTF>
-</plugin>
-</gazebo>
-<gazebo>
-<plugin name="gps_ground_truth_controller" filename="librobotnik_gazebo_ground_truth_odom.so">
-  <alwaysOn>true</alwaysOn>
-  <updateRate>50.0</updateRate>
-  <bodyName>gps_base_link</bodyName>
-  <frameName>gps_base_link_gt</frameName>
-  <worldBodyName>world</worldBodyName>
-  <worldFrameName>world</worldFrameName>
-  <topicName>odom_gt</topicName>
-  <gaussianNoise>0.01</gaussianNoise>
-  <xyzOffset>0.0 0 0</xyzOffset>
-  <rpyOffset>0 0 0</rpyOffset>
-  <applyOffset>False</applyOffset>
-  <broadcastTF>True</broadcastTF>
-</plugin>
-</gazebo>
+  <!-- Gazebo skid steering pluggins -->
+  <!-- xacro:skid_steering broadcastOdomTF="1"/ -->
+  <!-- WHEELS -->
+  <!-- Wheels -->
+  <xacro:front_wheel lr_prefix="left" fr_prefix="front"
+                     lr_reflect="1" fr_reflect="1" parent="base_link" />
+  <xacro:front_wheel lr_prefix="right" fr_prefix="front"
+                     lr_reflect="-1" fr_reflect="1" parent="base_link" />
+  <xacro:rear_wheel lr_prefix="left" fr_prefix="rear"
+                    lr_reflect="1" fr_reflect="-1" parent="base_link" />
+  <xacro:rear_wheel lr_prefix="right" fr_prefix="rear"
+                    lr_reflect="-1" fr_reflect="-1" parent="base_link" />
+  <!-- SENSORS -->
+  <xacro:sensor_benewake_ce30d prefix="front_3d_lidar" parent="base_link" gpu="true">
+      <origin xyz="2.155 0.0 0.236" rpy="0 0.24396 0"/>
+  </xacro:sensor_benewake_ce30d>
+  <xacro:sensor_rubedos_viper prefix="viper" parent="base_link">
+      <origin xyz="1.289 0.0 1.354" rpy="0 0.1745 0.0"/>
+  </xacro:sensor_rubedos_viper>
+  <xacro:sensor_imu_hector prefix="imu" parent="base_link">
+    <origin xyz="0.0 0.0 0.170" rpy="0 0 0"/>
+    <!--<origin xyz="0.917 0.0 0.170" rpy="0 0 0"/>-->
+  </xacro:sensor_imu_hector>
+  <xacro:sensor_gps prefix="gps" parent="base_link">
+    <origin xyz="0.0 0 1.5" rpy="0 0 0"/>
+  </xacro:sensor_gps>
 </robot>

Commit message: switched to 2d laser

File: rbcar_description/robots/rbcar.urdf.xacro (robot description, xacro)
@@ -44,10 +44,13 @@
                     lr_reflect="-1" fr_reflect="-1" parent="base_link" />
   <!-- SENSORS -->
-  <xacro:sensor_benewake_ce30d prefix="front_3d_lidar" parent="base_link" gpu="true">
+  <!--xacro:sensor_benewake_ce30d prefix="front_3d_lidar" parent="base_link" gpu="true">
       <origin xyz="2.155 0.0 0.236" rpy="0 0.24396 0"/>
-  </xacro:sensor_benewake_ce30d>
+  </xacro:sensor_benewake_ce30d-->
   <xacro:sensor_rubedos_viper prefix="viper" parent="base_link">
       <origin xyz="1.289 0.0 1.354" rpy="0 0.1745 0.0"/>
   </xacro:sensor_rubedos_viper>
+  <xacro:sensor_sick_s300 prefix="front_laser" parent="base_link" prefix_topic="front_laser" min_angle="-1.5" max_angle="1.5" gpu="false">
+      <origin xyz="2.2 0 0.3" rpy="0 0 0"/>
+  </xacro:sensor_sick_s300>
   <xacro:sensor_imu_hector prefix="imu" parent="base_link">
     <origin xyz="0.0 0.0 0.170" rpy="0 0 0"/>
