Commit message: description: added an elevator for the gps

File: rbcar_description/robots/rbcar.urdf.xacro (robot description, xacro)
@@ -2,61 +2,69 @@
   <robot name="rbcar"
     xmlns:xacro="http://wiki.ros.org/xacro">
-  <!-- ***************** -->
-  <!-- Imported elements -->
-  <!-- ***************** -->
-  <!-- First we import all posible elements defined in the urdf.xacro files. All these elements are defined as macro:xacros -->
-  <!-- Import Robotnik CAR base elements -->
-  <xacro:include filename="$(find rbcar_description)/urdf/bases/rbcar_base.urdf.xacro" />
-  <!-- Import Robotnik CAR wheels -->
-  <xacro:include filename="$(find rbcar_description)/urdf/wheels/suspension_wheel_v2.urdf.xacro" />
-  <!-- Import all available sensors -->
-  <xacro:include filename="$(find robotnik_sensors)/urdf/all_sensors.urdf.xacro" />
-  <!-- ***************** -->
-  <!-- Global parameters -->
-  <!-- ***************** -->
-  <xacro:property name="PI" value="3.1415926535897931"/>
-  <!-- Wheel parameters -->
-  <xacro:property name="wheel_offset_x" value="1.0" />    <!-- x,y,z in translation from base_link to the center of the wheel -->
-  <xacro:property name="wheel_offset_y" value="0.75" />
-  <xacro:property name="wheel_offset_z" value="0.0" />
-  <!-- Flag to select the high or low quality model -->
-  <xacro:property name="hq" value="true" />
-  <!-- *************** -->
-  <!-- Robots Elements -->
-  <!-- *************** -->
-  <!-- Here we create the robot elements using the xacro:macros imported at the beggining of this file -->
-  <!-- Summit XL base -->
-  <xacro:rbcar_base name="rbcar" publish_bf="true" hq="${hq}" />
-  <!-- Gazebo ros control pluggins -->
-  <xacro:ros_control/>
+	<!-- ***************** -->
+	<!-- Imported elements -->
+	<!-- ***************** -->
+	<!-- First we import all posible elements defined in the urdf.xacro files. All these elements are defined as macro:xacros -->
+	<!-- Import Robotnik CAR base elements -->
+	<xacro:include filename="$(find rbcar_description)/urdf/bases/rbcar_base.urdf.xacro" />
+	<!-- Import Robotnik CAR wheels -->
+	<xacro:include filename="$(find rbcar_description)/urdf/wheels/suspension_wheel_v2.urdf.xacro" />
+	<xacro:include filename="$(find rbcar_description)/urdf/structures/elevator.urdf.xacro" />
+	<!-- Import all available sensors -->
+	<xacro:include filename="$(find robotnik_sensors)/urdf/all_sensors.urdf.xacro" />
+	<!-- ***************** -->
+	<!-- Global parameters -->
+	<!-- ***************** -->
+	<xacro:property name="PI" value="3.1415926535897931"/>
+	<!-- Wheel parameters -->
+	<xacro:property name="wheel_offset_x" value="1.0" />    <!-- x,y,z in translation from base_link to the center of the wheel -->
+	<xacro:property name="wheel_offset_y" value="0.75" />
+	<xacro:property name="wheel_offset_z" value="0.0" />
+	<!-- Flag to select the high or low quality model -->
+	<xacro:property name="hq" value="true" />
+	<!-- *************** -->
+	<!-- Robots Elements -->
+	<!-- *************** -->
+	<!-- Here we create the robot elements using the xacro:macros imported at the beggining of this file -->
+	<!-- Summit XL base -->
+	<xacro:rbcar_base name="rbcar" publish_bf="true" hq="${hq}" />
+	<!-- Gazebo ros control pluggins -->
+	<xacro:ros_control/>
         <!-- xacro:omni_steering prefix="" publish_tf="true"/-->
-  <!-- Gazebo skid steering pluggins -->
-  <!-- xacro:skid_steering broadcastOdomTF="1"/ -->
-  <!-- WHEELS -->
-  <!-- Wheels -->
-  <xacro:front_wheel lr_prefix="left" fr_prefix="front"
-                     lr_reflect="1" fr_reflect="1" parent="base_link" />
-  <xacro:front_wheel lr_prefix="right" fr_prefix="front"
-                     lr_reflect="-1" fr_reflect="1" parent="base_link" />
-  <xacro:rear_wheel lr_prefix="left" fr_prefix="rear"
-                    lr_reflect="1" fr_reflect="-1" parent="base_link" />
-  <xacro:rear_wheel lr_prefix="right" fr_prefix="rear"
-                    lr_reflect="-1" fr_reflect="-1" parent="base_link" />
-  <!-- SENSORS -->
+	<!-- Gazebo skid steering pluggins -->
+	<!-- xacro:skid_steering broadcastOdomTF="1"/ -->
+	<!-- WHEELS -->
+    <!-- Wheels -->
+    <xacro:front_wheel lr_prefix="left" fr_prefix="front"
+                       lr_reflect="1" fr_reflect="1" parent="base_link" />
+    <xacro:front_wheel lr_prefix="right" fr_prefix="front"
+                       lr_reflect="-1" fr_reflect="1" parent="base_link" />
+    <xacro:rear_wheel lr_prefix="left" fr_prefix="rear"
+                      lr_reflect="1" fr_reflect="-1" parent="base_link" />
+    <xacro:rear_wheel lr_prefix="right" fr_prefix="rear"
+                      lr_reflect="-1" fr_reflect="-1" parent="base_link" />
+	<!-- SENSORS -->
   <!--xacro:sensor_benewake_ce30d prefix="front_3d_lidar" parent="base_link" gpu="true">
       <origin xyz="2.155 0.0 0.236" rpy="0 0.24396 0"/>
   </xacro:sensor_benewake_ce30d-->
   <xacro:sensor_rubedos_viper prefix="viper" parent="base_link">
-      <origin xyz="1.289 0.0 1.354" rpy="0 0.1745 0.0"/>
+    <origin xyz="1.289 0.0 1.354" rpy="0 0.1745 0.0"/>
   </xacro:sensor_rubedos_viper>
+	<xacro:sensor_imu_hector prefix="imu" parent="base_link">
+		<origin xyz="0.0 0.0 0.170" rpy="0 0 0"/>
+		<!--<origin xyz="0.917 0.0 0.170" rpy="0 0 0"/>-->
+	</xacro:sensor_imu_hector>
   <xacro:sensor_sick_s300 prefix="front_laser" parent="base_link" prefix_topic="front_laser" min_angle="-1.5" max_angle="1.5" gpu="false">
-      <origin xyz="2.2 0 0.3" rpy="0 0 0"/>
+    <origin xyz="2.2 0 0.3" rpy="0 0 0"/>
   </xacro:sensor_sick_s300>
-  <xacro:sensor_imu_hector prefix="imu" parent="base_link">
-    <origin xyz="0.0 0.0 0.170" rpy="0 0 0"/>
-    <!--<origin xyz="0.917 0.0 0.170" rpy="0 0 0"/>-->
-  </xacro:sensor_imu_hector>
-  <xacro:sensor_gps prefix="gps" parent="base_link" gps_latitude="$(arg gps_latitude)" gps_longitude="$(arg gps_longitude)">
-    <origin xyz="0.0 0 1.5" rpy="0 0 0"/>
-  </xacro:sensor_gps>
+	<xacro:sensor_gps prefix="gps" parent="base_link" gps_latitude="$(arg gps_latitude)" gps_longitude="$(arg gps_longitude)">
+		<origin xyz="0.0 0 1.5" rpy="0 0 0"/>
+		<!--<origin xyz="0.747 0 1.5" rpy="0 0 0"/>-->
+	</xacro:sensor_gps>
+  <xacro:elevator parent="base_link">
+		<origin xyz="0.0 0.0 0.6" rpy="0 0 0"/>
+	</xacro:elevator>
+  <xacro:sensor_axis prefix="front_ptz_camera" parent="elevator_link">
+    <origin xyz="0 0 0" rpy="0 0 0"/>
+  </xacro:sensor_axis>
 </robot>

File: rbcar_description/urdf/bases/rbcar_base.urdf.xacro (robot description, xacro)
@@ -57,5 +57,5 @@
        <origin xyz="0.917 0 0" rpy="0 0 0 " />
        <geometry>
-         <mesh filename="package://rbcar_description/meshes/bases/rbcar_chassis.stl"/>
+         <mesh filename="package://rbcar_description/meshes/bases/roborder_chassis.stl"/>
        </geometry>
     </collision>

Commit message: added melex model

File: rbcar_description/robots/rbcar.urdf.xacro (robot description, xacro)
@@ -42,5 +42,5 @@
                     lr_reflect="-1" fr_reflect="-1" parent="base_link" />
 	<!-- SENSORS -->
-    <xacro:sensor_sick_s3000 prefix="front_laser" parent="base_link">
+        <xacro:sensor_sick_s3000 prefix="front_laser" parent="base_link">
 		<origin xyz="1.58 0.0 0.0" rpy="0 0.0 0"/>
 	</xacro:sensor_sick_s3000>
@@ -48,4 +48,8 @@
 		<origin xyz="0.0 0.0 0.170" rpy="0 0 0"/>
 	</xacro:sensor_imu>
+	<xacro:sensor_gps prefix="gps" parent="base_link" gps_latitude="$(arg gps_latitude)" gps_longitude="$(arg gps_longitude)" >
+		<origin xyz="0.0 0 1.5" rpy="0 0 0"/>
+		<!--<origin xyz="0.747 0 1.5" rpy="0 0 0"/>-->
+	</xacro:sensor_gps>
 	<!--xacro:sensor_hokuyo_utm30lx name="hokuyo" parent="base_link">
 		<origin xyz="0.0 0.0 0.33" rpy="0 0 0"/>
@@ -59,7 +63,4 @@
 		<origin xyz="0.19 0 0.17" rpy="0 ${15*PI/180} 0"/>
 	</xacro:sensor_axis-->
-	<xacro:sensor_gps prefix="gps" parent="base_link">
-		<origin xyz="-0.17 0 1.5" rpy="0 0 0"/>
-	</xacro:sensor_gps>
 <!--
 	<xacro:sensor_asus_xtion_pro name="xtion_pro" parent="base_link">
@@ -77,10 +78,10 @@
 	</xacro:sensor_fotonic>
 -->
-    <xacro:elevator parent="base_link">
+    <!--xacro:elevator parent="base_link">
 		<origin xyz="0.0 0.0 0.6" rpy="0 0 0"/>
-	</xacro:elevator>
-    <xacro:sensor_axis prefix="front_ptz_camera" parent="elevator_link" far="300" near="0.08">
+    </xacro:elevator-->
+    <!--xacro:sensor_axis prefix="front_ptz_camera" parent="elevator_link" far="300" near="0.08">
             <origin xyz="0 0 0" rpy="0 0 0"/>
-    </xacro:sensor_axis>
+    </xacro:sensor_axis-->
 <gazebo>
 <plugin name="ground_truth_controller" filename="librobotnik_gazebo_ground_truth_odom.so">

Commit message: modified the tfs to use the robot_ prefix

File: rbcar_description/robots/rbcar.urdf.xacro (robot description, xacro)
@@ -1,4 +1,5 @@
 <?xml version="1.0"?>
-<robot name="rbcar" xmlns:xacro="http://www.ros.org/wiki/xacro">
+<robot name="rbcar"
+	xmlns:xacro="http://www.ros.org/wiki/xacro">
 	<!-- ***************** -->
 	<!-- Imported elements -->
@@ -15,6 +16,8 @@
 	<!-- ***************** -->
 	<xacro:property name="PI" value="3.1415926535897931"/>
+	<xacro:property name="robot_prefix" value="robot_" />
 	<!-- Wheel parameters -->
-	<xacro:property name="wheel_offset_x" value="1.0" />    <!-- x,y,z in translation from base_link to the center of the wheel -->
+	<xacro:property name="wheel_offset_x" value="1.0" />
+	<!-- x,y,z in translation from base_link to the center of the wheel -->
 	<xacro:property name="wheel_offset_y" value="0.75" />
 	<xacro:property name="wheel_offset_z" value="0.0" />
@@ -25,6 +28,6 @@
 	<!-- *************** -->
 	<!-- Here we create the robot elements using the xacro:macros imported at the beggining of this file -->
-	<!-- Summit XL base -->
-	<xacro:rbcar_base name="rbcar" publish_bf="true" hq="${hq}" />
+	<!-- Rbcar base -->
+	<xacro:rbcar_base name="rbcar" publish_bf="true" hq="${hq}" prefix="${robot_prefix}"/>
 	<!-- Gazebo ros control pluggins -->
 	<xacro:ros_control/>
@@ -32,20 +35,16 @@
 	<!-- xacro:skid_steering broadcastOdomTF="1"/ -->
 	<!-- WHEELS -->
-  	<xacro:front_wheel lr_prefix="left" fr_prefix="front"
-                     lr_reflect="1" fr_reflect="1" parent="base_link" />
- 	 <xacro:front_wheel lr_prefix="right" fr_prefix="front"
-                     lr_reflect="-1" fr_reflect="1" parent="base_link" />
-  	<xacro:rear_wheel lr_prefix="left" fr_prefix="rear"
-                    lr_reflect="1" fr_reflect="-1" parent="base_link" />
-  	<xacro:rear_wheel lr_prefix="right" fr_prefix="rear"
-                    lr_reflect="-1" fr_reflect="-1" parent="base_link" />
+	<xacro:front_wheel lr_prefix="left" fr_prefix="front" lr_reflect="1" fr_reflect="1" parent="${robot_prefix}base_link" prefix="${robot_prefix}"/>
+	<xacro:front_wheel lr_prefix="right" fr_prefix="front" lr_reflect="-1" fr_reflect="1" parent="${robot_prefix}base_link" prefix="${robot_prefix}"/>
+	<xacro:rear_wheel lr_prefix="left" fr_prefix="rear" lr_reflect="1" fr_reflect="-1" parent="${robot_prefix}base_link" prefix="${robot_prefix}"/>
+	<xacro:rear_wheel lr_prefix="right" fr_prefix="rear" lr_reflect="-1" fr_reflect="-1" parent="${robot_prefix}base_link" prefix="${robot_prefix}"/>
 	<!-- SENSORS -->
-        <xacro:sensor_sick_s3000 prefix="front_laser" parent="base_link">
+	<xacro:sensor_sick_s3000 prefix="${robot_prefix}front_laser" parent="${robot_prefix}base_link">
 		<origin xyz="1.58 0.0 0.0" rpy="0 0.0 0"/>
 	</xacro:sensor_sick_s3000>
-	<xacro:sensor_imu prefix="imu" parent="base_link">
+	<xacro:sensor_imu prefix="${robot_prefix}imu" parent="${robot_prefix}base_link">
 		<origin xyz="0.0 0.0 0.170" rpy="0 0 0"/>
 	</xacro:sensor_imu>
-	<xacro:sensor_gps prefix="gps" parent="base_link" gps_latitude="$(arg gps_latitude)" gps_longitude="$(arg gps_longitude)" >
+	<xacro:sensor_gps prefix="${robot_prefix}gps" parent="${robot_prefix}base_link" gps_latitude="$(arg gps_latitude)" gps_longitude="$(arg gps_longitude)">
 		<origin xyz="0.0 0 1.5" rpy="0 0 0"/>
 		<!--<origin xyz="0.747 0 1.5" rpy="0 0 0"/>-->
@@ -76,35 +75,35 @@
             <origin xyz="0 0 0" rpy="0 0 0"/>
     	</xacro:sensor_axis-->
-<gazebo>
-<plugin name="ground_truth_controller" filename="librobotnik_gazebo_ground_truth_odom.so">
-  <alwaysOn>true</alwaysOn>
-  <updateRate>50.0</updateRate>
-  <bodyName>base_link</bodyName>
-  <frameName>base_link_gt</frameName>
-  <worldBodyName>world</worldBodyName>
-  <worldFrameName>world</worldFrameName>
-  <topicName>odom_gt</topicName>
-  <gaussianNoise>0.01</gaussianNoise>
-  <xyzOffset>0.0 0 0</xyzOffset>
-  <rpyOffset>0 0 0</rpyOffset>
-  <applyOffset>False</applyOffset>
-  <broadcastTF>True</broadcastTF>
-</plugin>
-</gazebo>
-<gazebo>
-<plugin name="gps_ground_truth_controller" filename="librobotnik_gazebo_ground_truth_odom.so">
-  <alwaysOn>true</alwaysOn>
-  <updateRate>50.0</updateRate>
-  <bodyName>gps_base_link</bodyName>
-  <frameName>gps_base_link_gt</frameName>
-  <worldBodyName>world</worldBodyName>
-  <worldFrameName>world</worldFrameName>
-  <topicName>odom_gt</topicName>
-  <gaussianNoise>0.01</gaussianNoise>
-  <xyzOffset>0.0 0 0</xyzOffset>
-  <rpyOffset>0 0 0</rpyOffset>
-  <applyOffset>False</applyOffset>
-  <broadcastTF>True</broadcastTF>
-</plugin>
-</gazebo>
+	<gazebo>
+		<plugin name="ground_truth_controller" filename="librobotnik_gazebo_ground_truth_odom.so">
+			<alwaysOn>true</alwaysOn>
+			<updateRate>50.0</updateRate>
+			<bodyName>base_link</bodyName>
+			<frameName>base_link_gt</frameName>
+			<worldBodyName>world</worldBodyName>
+			<worldFrameName>world</worldFrameName>
+			<topicName>odom_gt</topicName>
+			<gaussianNoise>0.01</gaussianNoise>
+			<xyzOffset>0.0 0 0</xyzOffset>
+			<rpyOffset>0 0 0</rpyOffset>
+			<applyOffset>False</applyOffset>
+			<broadcastTF>True</broadcastTF>
+		</plugin>
+	</gazebo>
+	<gazebo>
+		<plugin name="gps_ground_truth_controller" filename="librobotnik_gazebo_ground_truth_odom.so">
+			<alwaysOn>true</alwaysOn>
+			<updateRate>50.0</updateRate>
+			<bodyName>gps_base_link</bodyName>
+			<frameName>gps_base_link_gt</frameName>
+			<worldBodyName>world</worldBodyName>
+			<worldFrameName>world</worldFrameName>
+			<topicName>odom_gt</topicName>
+			<gaussianNoise>0.01</gaussianNoise>
+			<xyzOffset>0.0 0 0</xyzOffset>
+			<rpyOffset>0 0 0</rpyOffset>
+			<applyOffset>False</applyOffset>
+			<broadcastTF>True</broadcastTF>
+		</plugin>
+	</gazebo>
 </robot>

Commit message: rbcar_description: Add velodyne to rbcar.urdf.xacro

File: rbcar_description/robots/rbcar.urdf.xacro (robot description, xacro)
@@ -48,4 +48,7 @@
       <origin xyz="2.155 0.0 0.236" rpy="0 0.24396 0"/>
   </xacro:sensor_benewake_ce30d-->
+  <xacro:sensor_velodyne_vlp16 prefix="front_3d_lidar" parent="base_link" range_min="0.8" range_max="31.0" gpu="false">
+      <origin xyz="2.155 0.0 0.236" rpy="0 0.24396 0"/>
+  </xacro:sensor_velodyne_vlp16>
   <xacro:sensor_rubedos_viper prefix="viper" parent="base_link">
     <origin xyz="1.289 0.0 1.354" rpy="0 0.1745 0.0"/>
@@ -55,7 +58,7 @@
 		<!--<origin xyz="0.917 0.0 0.170" rpy="0 0 0"/>-->
 	</xacro:sensor_imu_hector>
-  <xacro:sensor_sick_s300 prefix="front_laser" parent="base_link" prefix_topic="front_laser" min_angle="-1.5" max_angle="1.5" gpu="false">
+  <!--xacro:sensor_sick_s300 prefix="front_laser" parent="base_link" prefix_topic="front_laser" min_angle="-1.5" max_angle="1.5" gpu="false">
     <origin xyz="2.2 0 0.3" rpy="0 0 0"/>
-  </xacro:sensor_sick_s300>
+  </xacro:sensor_sick_s300-->
 	<xacro:sensor_gps prefix="gps" parent="base_link" gps_latitude="$(arg gps_latitude)" gps_longitude="$(arg gps_longitude)">
 		<origin xyz="0.0 0 1.5" rpy="0 0 0"/>

Commit message: added wheelbase param

File: rbcar_description/robots/rbcar.urdf.xacro (robot description, xacro)
@@ -24,4 +24,5 @@
 	<!-- Flag to select the high or low quality model -->
 	<xacro:property name="hq" value="true" />
+	<xacro:property name="wheelbase" value="1.63" />
 	<!-- *************** -->
 	<!-- Robots Elements -->
@@ -29,5 +30,5 @@
 	<!-- Here we create the robot elements using the xacro:macros imported at the beggining of this file -->
 	<!-- Rbcar base -->
-	<xacro:rbcar_base name="rbcar" publish_bf="true" hq="${hq}" prefix="${robot_prefix}"/>
+	<xacro:rbcar_base name="rbcar" publish_bf="true" hq="${hq}" prefix="${robot_prefix}" wheelbase="${wheelbase}"/>
 	<!-- Gazebo ros control pluggins -->
 	<xacro:ros_control/>
