Commit message: description: Use-prefix compability

File: rbcar_description/robots/rbcar.urdf.xacro (robot description, xacro)
@@ -10,5 +10,4 @@
 	<!-- Import Robotnik CAR wheels -->
 	<xacro:include filename="$(find rbcar_description)/urdf/wheels/suspension_wheel_v2.urdf.xacro" />
-	<xacro:include filename="$(find rbcar_description)/urdf/structures/elevator.urdf.xacro" />
 	<!-- Import all available sensors -->
 	<xacro:include filename="$(find robotnik_sensors)/urdf/all_sensors.urdf.xacro" />
@@ -23,4 +22,7 @@
 	<!-- Flag to select the high or low quality model -->
 	<xacro:property name="hq" value="true" />
+	<xacro:arg name="prefix" default="robot_"/>
+	<xacro:arg name="gps_longitude" default="39.5091874"/>
+	<xacro:arg name="gps_latitude" default="-0.4637371"/>
 	<!-- *************** -->
 	<!-- Robots Elements -->
@@ -28,46 +30,28 @@
 	<!-- Here we create the robot elements using the xacro:macros imported at the beggining of this file -->
 	<!-- Summit XL base -->
-	<xacro:rbcar_base name="rbcar" publish_bf="true" hq="${hq}" />
+	<xacro:rbcar_base name="rbcar" prefix="$(arg prefix)" publish_bf="true" hq="${hq}" />
 	<!-- Gazebo ros control pluggins -->
 	<xacro:ros_control/>
-        <!-- xacro:omni_steering prefix="" publish_tf="true"/-->
-	<!-- Gazebo skid steering pluggins -->
-	<!-- xacro:skid_steering broadcastOdomTF="1"/ -->
-	<!-- WHEELS -->
-    <!-- Wheels -->
-    <xacro:front_wheel lr_prefix="left" fr_prefix="front"
-                       lr_reflect="1" fr_reflect="1" parent="base_link" />
-    <xacro:front_wheel lr_prefix="right" fr_prefix="front"
-                       lr_reflect="-1" fr_reflect="1" parent="base_link" />
-    <xacro:rear_wheel lr_prefix="left" fr_prefix="rear"
-                      lr_reflect="1" fr_reflect="-1" parent="base_link" />
-    <xacro:rear_wheel lr_prefix="right" fr_prefix="rear"
-                      lr_reflect="-1" fr_reflect="-1" parent="base_link" />
-	<!-- SENSORS -->
-  <!--xacro:sensor_benewake_ce30d prefix="front_3d_lidar" parent="base_link" gpu="true">
-      <origin xyz="2.155 0.0 0.236" rpy="0 0.24396 0"/>
-  </xacro:sensor_benewake_ce30d-->
-  <xacro:sensor_velodyne_vlp16 prefix="front_3d_lidar" parent="base_link" range_min="0.8" range_max="31.0" gpu="false">
-      <origin xyz="2.155 0.0 0.236" rpy="0 0.24396 0"/>
-  </xacro:sensor_velodyne_vlp16>
-  <xacro:sensor_rubedos_viper prefix="viper" parent="base_link">
-    <origin xyz="1.289 0.0 1.354" rpy="0 0.1745 0.0"/>
-  </xacro:sensor_rubedos_viper>
-	<xacro:sensor_imu_hector prefix="imu" parent="base_link">
+	<!-- Wheels -->
+	<xacro:front_wheel lr_prefix="$(arg prefix)left" fr_prefix="front"
+					 lr_reflect="1" fr_reflect="1" parent="$(arg prefix)base_link" />
+	<xacro:front_wheel lr_prefix="$(arg prefix)right" fr_prefix="front"
+					 lr_reflect="-1" fr_reflect="1" parent="$(arg prefix)base_link" />
+	<xacro:rear_wheel lr_prefix="$(arg prefix)left" fr_prefix="rear"
+					lr_reflect="1" fr_reflect="-1" parent="$(arg prefix)base_link" />
+	<xacro:rear_wheel lr_prefix="$(arg prefix)right" fr_prefix="rear"
+					lr_reflect="-1" fr_reflect="-1" parent="$(arg prefix)base_link" />
+	<xacro:sensor_rslidar_16 prefix="$(arg prefix)top_3d_laser" parent="$(arg prefix)base_link">
+	  <origin xyz="1.0 0.0 1.5" rpy="0 0.24396 0"/>
+	</xacro:sensor_rslidar_16>
+	<xacro:sensor_imu_hector prefix="$(arg prefix)imu" parent="$(arg prefix)base_link">
 		<origin xyz="0.0 0.0 0.170" rpy="0 0 0"/>
 		<!--<origin xyz="0.917 0.0 0.170" rpy="0 0 0"/>-->
 	</xacro:sensor_imu_hector>
-  <!--xacro:sensor_sick_s300 prefix="front_laser" parent="base_link" prefix_topic="front_laser" min_angle="-1.5" max_angle="1.5" gpu="false">
-    <origin xyz="2.2 0 0.3" rpy="0 0 0"/>
-  </xacro:sensor_sick_s300-->
-	<xacro:sensor_gps prefix="gps" parent="base_link" gps_latitude="$(arg gps_latitude)" gps_longitude="$(arg gps_longitude)">
+	<xacro:sensor_sick_outdoorscan3 prefix="$(arg prefix)front_laser" parent="$(arg prefix)base_link" prefix_topic="front_laser" min_angle="-1.5" max_angle="1.5" gpu="false">
+		<origin xyz="2.2 0 0.3" rpy="0 0 0"/>
+	</xacro:sensor_sick_outdoorscan3>
+	<xacro:sensor_gps prefix="$(arg prefix)gps" parent="$(arg prefix)base_link" gps_latitude="$(arg gps_latitude)" gps_longitude="$(arg gps_longitude)">
 		<origin xyz="0.0 0 1.5" rpy="0 0 0"/>
-		<!--<origin xyz="0.747 0 1.5" rpy="0 0 0"/>-->
 	</xacro:sensor_gps>
-  <xacro:elevator parent="base_link">
-		<origin xyz="0.0 0.0 0.6" rpy="0 0 0"/>
-	</xacro:elevator>
-  <xacro:sensor_axis prefix="front_ptz_camera" parent="elevator_link">
-    <origin xyz="0 0 0" rpy="0 0 0"/>
-  </xacro:sensor_axis>
 </robot>

File: rbcar_description/urdf/bases/rbcar_base.urdf.xacro (robot description, xacro)
@@ -2,5 +2,5 @@
 <robot name="rbcar" xmlns:xacro="http://wiki.ros.org/xacro">
   <xacro:include filename="$(find rbcar_description)/urdf/bases/rbcar_base.gazebo.xacro" />
-  <xacro:macro name="rbcar_base" params="name publish_bf hq">
+  <xacro:macro name="rbcar_base" params="prefix name publish_bf hq">
   <!-- Robot mechanical and motor parameters -->
   <xacro:property name="PI" value="3.1415926535897931"/>
@@ -9,5 +9,5 @@
   <!-- BASE FOOTPRINT -->
   <xacro:if value="${publish_bf}">
-    <link name="base_footprint">
+    <link name="${prefix}base_footprint">
       <visual>
           <origin xyz="0 0 0" rpy="0 0 0" />
@@ -25,12 +25,12 @@
 -->
     </link>
-    <joint name="base_footprint_joint" type="fixed">
+    <joint name="${prefix}base_footprint_joint" type="fixed">
       <origin xyz="0 0 ${clearance}" rpy="0 0 0" />  <!-- height is the clearance -->
-      <parent link="base_footprint"/>
-      <child link="base_link" />
+      <parent link="${prefix}base_footprint"/>
+      <child link="${prefix}base_link" />
     </joint>
   </xacro:if>
   <!-- BASE_LINK -->
-  <link name="base_link">
+  <link name="${prefix}base_link">
     <inertial>
       <mass value="125.0" />

File: rbcar_description/urdf/wheels/suspension_wheel_v2.urdf.xacro (robot description, xacro)
@@ -15,5 +15,5 @@
        from a U joint to the corresponding hex hub. wheel_travel is the
        vertical wheel travel. -->
-  <xacro:property name="wheelbase" value="1.83323"/>
+  <xacro:property name="wheelbase" value="1.86"/>
   <!--xacro:property name="hex_hub_dist" value="1.2385"/-->  <!-- 1.127 0.742 0.900 check -->
   <xacro:property name="axle_length" value="0.120"/>
@@ -122,5 +122,5 @@
       <parent link="${lr_prefix}_${fr_prefix}_axle_carrier"/>
       <child link="${lr_prefix}_${fr_prefix}_wheel"/>
-      <origin rpy="${degrees_90} 0 ${degrees_180}"/>
+      <origin rpy="-${degrees_90} 0 0"/>
       <axis xyz="0 0 1"/>
       <limit effort="${axle_eff_limit}" velocity="${axle_vel_limit}"/>
@@ -142,14 +142,7 @@
     <link name="${lr_prefix}_${fr_prefix}_wheel">
       <visual>
-        <xacro:if value="${lr_prefix=='left'}">
           <origin xyz="0
                        0
-                       ${lr_reflect * (axle_length - (tire_width / 2 - hex_hub_depth))}" rpy = "${degrees_90} 0 ${degrees_180}"/>
-        </xacro:if>
-        <xacro:if value="${lr_prefix=='right'}">
-          <origin xyz="0
-                       0
-                       ${lr_reflect * (axle_length - (tire_width / 2 - hex_hub_depth))}" rpy = "-${degrees_90} 0 ${degrees_180}"/>
-        </xacro:if>
+                       ${lr_reflect * (axle_length - (tire_width / 2 - hex_hub_depth))}" rpy = "${lr_reflect * degrees_90} 0 ${degrees_180}"/>
         <geometry>
           <!--cylinder radius="${tire_dia / 2}" length="${tire_width}"/-->

Commit message: description: update default sensors positions

File: rbcar_description/robots/rbcar.urdf.xacro (robot description, xacro)
@@ -43,15 +43,14 @@
 					lr_reflect="-1" fr_reflect="-1" parent="$(arg prefix)base_link" />
 	<xacro:sensor_rslidar_16 prefix="$(arg prefix)top_3d_laser" parent="$(arg prefix)base_link">
-	  <origin xyz="1.0 0.0 1.5" rpy="0 0.24396 0"/>
+	  <origin xyz="1.163 0.0 1.602" rpy="0 0.2637 0"/>
 	</xacro:sensor_rslidar_16>
 	<xacro:sensor_imu_hector prefix="$(arg prefix)imu" parent="$(arg prefix)base_link">
-		<origin xyz="0.0 0.0 0.170" rpy="0 0 0"/>
-		<!--<origin xyz="0.917 0.0 0.170" rpy="0 0 0"/>-->
+		<origin xyz="0.319 0.018 0.676" rpy="0 0 0"/>
 	</xacro:sensor_imu_hector>
 	<xacro:sensor_sick_outdoorscan3 prefix="$(arg prefix)front_laser" parent="$(arg prefix)base_link" prefix_topic="front_laser" min_angle="-1.5" max_angle="1.5" gpu="false">
-		<origin xyz="2.2 0 0.3" rpy="0 0 0"/>
+		<origin xyz="2.101 0 0.206" rpy="0 0 0"/>
 	</xacro:sensor_sick_outdoorscan3>
 	<xacro:sensor_gps prefix="$(arg prefix)gps" parent="$(arg prefix)base_link" gps_latitude="$(arg gps_latitude)" gps_longitude="$(arg gps_longitude)">
-		<origin xyz="0.0 0 1.5" rpy="0 0 0"/>
+		<origin xyz="0.491 0 1.503" rpy="0 0 0"/>
 	</xacro:sensor_gps>
 </robot>

File: rbcar_description/urdf/wheels/suspension_wheel_v2.urdf.xacro (robot description, xacro)
@@ -15,5 +15,5 @@
        from a U joint to the corresponding hex hub. wheel_travel is the
        vertical wheel travel. -->
-  <xacro:property name="wheelbase" value="1.86"/>
+  <xacro:property name="wheelbase" value="1.83"/>
   <!--xacro:property name="hex_hub_dist" value="1.2385"/-->  <!-- 1.127 0.742 0.900 check -->
   <xacro:property name="axle_length" value="0.120"/>

Commit message: description: Add rear axle into std model

File: rbcar_description/robots/rbcar.urdf.xacro (robot description, xacro)
@@ -10,4 +10,5 @@
 	<!-- Import Robotnik CAR wheels -->
 	<xacro:include filename="$(find rbcar_description)/urdf/wheels/suspension_wheel_v2.urdf.xacro" />
+	<xacro:include filename="$(find rbcar_description)/urdf/wheels/rear_axle.urdf.xacro" />
 	<!-- Import all available sensors -->
 	<xacro:include filename="$(find robotnik_sensors)/urdf/all_sensors.urdf.xacro" />
@@ -42,4 +43,7 @@
 	<xacro:rear_wheel lr_prefix="$(arg prefix)right" fr_prefix="rear"
 					lr_reflect="-1" fr_reflect="-1" parent="$(arg prefix)base_link" />
+    <xacro:rear_axle prefix="$(arg prefix)rear_axle" parent="$(arg prefix)base_link">
+	  <origin xyz="0 0.0 0" rpy="1.57079633 0 3.14159265"/>
+    </xacro:rear_axle>
 	<xacro:sensor_rslidar_16 prefix="$(arg prefix)top_3d_laser" parent="$(arg prefix)base_link">
 	  <origin xyz="1.163 0.0 1.602" rpy="0 0.2637 0"/>

File: rbcar_description/urdf/wheels/rear_axle.urdf.xacro (robot description, xacro)
@@ -3,8 +3,7 @@
   <xacro:macro name="rear_axle" params="prefix parent *origin">
     <joint name="${prefix}_joint" type="continuous">
-      <parent link="base_link"/>
+      <parent link="${parent}"/>
       <child link="${prefix}"/>
       <xacro:insert_block name="origin" />
-      <!--origin xyz="-0.91131 0 0" rpy="1.57079633 0 3.14159265"/-->
       <axis xyz="0 0 1"/>
       <limit effort="600" velocity="1000"/>

Commit message: description: update default urdf model

File: rbcar_description/robots/rbcar.urdf.xacro (robot description, xacro)
@@ -9,5 +9,5 @@
 	<xacro:include filename="$(find rbcar_description)/urdf/bases/rbcar_base.urdf.xacro" />
 	<!-- Import Robotnik CAR wheels -->
-	<xacro:include filename="$(find rbcar_description)/urdf/wheels/suspension_wheel_v2.urdf.xacro" />
+	<xacro:include filename="$(find rbcar_description)/urdf/wheels/suspension_wheel_v3.urdf.xacro" />
 	<xacro:include filename="$(find rbcar_description)/urdf/wheels/rear_axle.urdf.xacro" />
 	<!-- Import all available sensors -->
@@ -43,7 +43,7 @@
 	<xacro:rear_wheel lr_prefix="$(arg prefix)right" fr_prefix="rear"
 					lr_reflect="-1" fr_reflect="-1" parent="$(arg prefix)base_link" />
-    <xacro:rear_axle prefix="$(arg prefix)rear_axle" parent="$(arg prefix)base_link">
-	  <origin xyz="0 0.0 0" rpy="1.57079633 0 3.14159265"/>
-    </xacro:rear_axle>
+  <xacro:rear_axle prefix="$(arg prefix)rear_axle" parent="$(arg prefix)base_link">
+    <origin xyz="0 0.0 0" rpy="1.57079633 0 3.14159265"/>
+  </xacro:rear_axle>
 	<xacro:sensor_rslidar_16 prefix="$(arg prefix)top_3d_laser" parent="$(arg prefix)base_link">
 	  <origin xyz="1.163 0.0 1.602" rpy="0 0.2637 0"/>
@@ -53,5 +53,5 @@
 	</xacro:sensor_imu_hector>
 	<xacro:sensor_sick_outdoorscan3 prefix="$(arg prefix)front_laser" parent="$(arg prefix)base_link" prefix_topic="front_laser" min_angle="-1.5" max_angle="1.5" gpu="false">
-		<origin xyz="2.101 0 0.206" rpy="0 0 0"/>
+		<origin xyz="2.350 0 0.206" rpy="0 0 0"/>
 	</xacro:sensor_sick_outdoorscan3>
 	<xacro:sensor_gps prefix="$(arg prefix)gps" parent="$(arg prefix)base_link" gps_latitude="$(arg gps_latitude)" gps_longitude="$(arg gps_longitude)">

File: rbcar_description/urdf/wheels/rear_axle.urdf.xacro (robot description, xacro)
@@ -25,5 +25,5 @@
         <origin xyz="0 0 0"/>
         <geometry>
-          <cylinder length="0.2" radius="0.317"/>
+          <cylinder length="0.05" radius="0.15"/>
         </geometry>
         <material name="tire_mat"/>

File: rbcar_description/urdf/wheels/suspension_wheel_v3.urdf.xacro (robot description, xacro)
@@ -146,10 +146,10 @@
     <link name="${lr_prefix}_${fr_prefix}_wheel">
       <visual>
-        <xacro:if value="${lr_prefix=='left'}">
+        <xacro:if value="${lr_prefix.endswith('left')}">
           <origin xyz="0
                        0
                        ${lr_reflect * (axle_length - (tire_width / 2 - hex_hub_depth))}" rpy = "${degrees_90} 0 ${degrees_180}"/>
         </xacro:if>
-        <xacro:if value="${lr_prefix=='right'}">
+        <xacro:if value="${lr_prefix.endswith('right')}">
           <origin xyz="0
                        0
