Commit message: Update rbcar models

File: rbcar_description/robots/rbcar.urdf.xacro (robot description, xacro)
@@ -9,8 +9,9 @@
 	<xacro:include filename="$(find rbcar_description)/urdf/bases/rbcar_base.urdf.xacro" />
 	<!-- Import Robotnik CAR wheels -->
-	<xacro:include filename="$(find rbcar_description)/urdf/wheels/suspension_wheel_v2.urdf.xacro" />
-	<xacro:include filename="$(find rbcar_description)/urdf/wheels/rear_axle.urdf.xacro" />
+	<xacro:include filename="$(find rbcar_description)/urdf/wheels/suspension_wheel_v3.urdf.xacro" />
 	<!-- Import all available sensors -->
+	<xacro:include filename="$(find rbcar_description)/urdf/structures/elevator.urdf.xacro" />
 	<xacro:include filename="$(find robotnik_sensors)/urdf/all_sensors.urdf.xacro" />
+  	<xacro:include filename="$(find robotnik_sensors)/urdf/utils/inertia.urdf.xacro" />
 	<!-- ***************** -->
 	<!-- Global parameters -->
@@ -18,12 +19,12 @@
 	<xacro:property name="PI" value="3.1415926535897931"/>
 	<!-- Wheel parameters -->
-	<xacro:property name="wheel_offset_x" value="1.0" />    <!-- x,y,z in translation from base_link to the center of the wheel -->
-	<xacro:property name="wheel_offset_y" value="0.75" />
+	<xacro:property name="wheel_offset_x" value="0.91131" />    <!-- x,y,z in translation from base_link to the center of the wheel -->
+	<xacro:property name="wheel_offset_y" value="0.62124" />
 	<xacro:property name="wheel_offset_z" value="0.0" />
 	<!-- Flag to select the high or low quality model -->
 	<xacro:property name="hq" value="true" />
 	<xacro:arg name="prefix" default="robot_"/>
-	<xacro:arg name="gps_longitude" default="39.5091874"/>
-	<xacro:arg name="gps_latitude" default="-0.4637371"/>
+	<xacro:arg name="gps_longitude" default="39.551218"/>
+	<xacro:arg name="gps_latitude" default="-0.467738"/>
 	<xacro:arg name="gpu" default="true"/>
 	<!-- *************** -->
@@ -31,22 +32,20 @@
 	<!-- *************** -->
 	<!-- Here we create the robot elements using the xacro:macros imported at the beggining of this file -->
-	<!-- Summit XL base -->
+	<!-- Rbcar base -->
 	<xacro:rbcar_base name="rbcar" prefix="$(arg prefix)" publish_bf="true" hq="${hq}" />
 	<!-- Gazebo ros control pluggins -->
 	<xacro:ros_control/>
 	<!-- Wheels -->
-	<xacro:front_wheel lr_prefix="$(arg prefix)left" fr_prefix="front"
-					 lr_reflect="1" fr_reflect="1" parent="$(arg prefix)base_link" />
-	<xacro:front_wheel lr_prefix="$(arg prefix)right" fr_prefix="front"
-					 lr_reflect="-1" fr_reflect="1" parent="$(arg prefix)base_link" />
-	<xacro:rear_wheel lr_prefix="$(arg prefix)left" fr_prefix="rear"
-					lr_reflect="1" fr_reflect="-1" parent="$(arg prefix)base_link" />
-	<xacro:rear_wheel lr_prefix="$(arg prefix)right" fr_prefix="rear"
-					lr_reflect="-1" fr_reflect="-1" parent="$(arg prefix)base_link" />
-    <xacro:rear_axle prefix="$(arg prefix)rear_axle" parent="$(arg prefix)base_link">
-	  <origin xyz="0 0.0 0" rpy="1.57079633 0 3.14159265"/>
-    </xacro:rear_axle>
-	<xacro:sensor_rslidar_16 prefix="$(arg prefix)top_3d_laser" parent="$(arg prefix)base_link"  gpu="$(arg gpu)">
-	  <origin xyz="1.163 0.0 1.602" rpy="0 0.2637 0"/>
+  	<xacro:front_wheel prefix="$(arg prefix)" lr_prefix="left" fr_prefix="front"
+                     lr_reflect="1" fr_reflect="1" parent="$(arg prefix)base_link" />
+  	<xacro:front_wheel prefix="$(arg prefix)" lr_prefix="right" fr_prefix="front"
+                     lr_reflect="-1" fr_reflect="1" parent="$(arg prefix)base_link" />
+  	<xacro:rear_wheel prefix="$(arg prefix)" lr_prefix="left" fr_prefix="rear"
+                    lr_reflect="1" fr_reflect="-1" parent="$(arg prefix)base_link" />
+  	<xacro:rear_wheel prefix="$(arg prefix)" lr_prefix="right" fr_prefix="rear"
+                    lr_reflect="-1" fr_reflect="-1" parent="$(arg prefix)base_link" />
+	<!-- SENSORS -->
+	<xacro:sensor_rslidar_16 prefix="$(arg prefix)top_3d_laser" parent="$(arg prefix)base_link"  gpu="$(arg gpu)" prefix_topic="top_3d_laser">
+	  <origin xyz="1.163 0.0 1.602" rpy="0 0 0"/>
 	</xacro:sensor_rslidar_16>
 	<xacro:sensor_imu_hector prefix="$(arg prefix)imu" parent="$(arg prefix)base_link">
@@ -54,8 +53,41 @@
 	</xacro:sensor_imu_hector>
 	<xacro:sensor_sick_outdoorscan3 prefix="$(arg prefix)front_laser" parent="$(arg prefix)base_link" prefix_topic="front_laser" min_angle="-1.5" max_angle="1.5" gpu="$(arg gpu)">
-		<origin xyz="2.101 0 0.206" rpy="0 0 0"/>
+		<origin xyz="2.15679 0 0.05433" rpy="0 0 0"/>
 	</xacro:sensor_sick_outdoorscan3>
 	<xacro:sensor_gps prefix="$(arg prefix)gps" parent="$(arg prefix)base_link" gps_latitude="$(arg gps_latitude)" gps_longitude="$(arg gps_longitude)">
 		<origin xyz="0.491 0 1.503" rpy="0 0 0"/>
 	</xacro:sensor_gps>
+<!--Gazebo plugins-->
+<gazebo>
+	<plugin name="ground_truth_controller" filename="librobotnik_gazebo_ground_truth_odom.so">
+		<alwaysOn>true</alwaysOn>
+		<updateRate>50.0</updateRate>
+		<bodyName>$(arg prefix)base_link</bodyName>
+		<frameName>base_footprint_gt</frameName>
+		<worldBodyName>world</worldBodyName>
+		<worldFrameName>$(arg prefix)odom</worldFrameName>
+		<topicName>odom_gt</topicName>
+		<gaussianNoise>0.01</gaussianNoise>
+		<xyzOffset>0.0 0 0</xyzOffset>
+		<rpyOffset>0 0 0</rpyOffset>
+		<applyOffset>False</applyOffset>
+		<broadcastTF>True</broadcastTF>
+	</plugin>
+</gazebo>
+<gazebo>
+	<plugin name="gps_ground_truth_controller" filename="librobotnik_gazebo_ground_truth_odom.so">
+		<alwaysOn>true</alwaysOn>
+		<updateRate>50.0</updateRate>
+		<bodyName>$(arg prefix)gps_base_link</bodyName>
+		<frameName>gps_base_link_gt</frameName>
+		<worldBodyName>world</worldBodyName>
+		<worldFrameName>world</worldFrameName>
+		<topicName>odom_gt</topicName>
+		<gaussianNoise>0.01</gaussianNoise>
+		<xyzOffset>0.0 0 0</xyzOffset>
+		<rpyOffset>0 0 0</rpyOffset>
+		<applyOffset>False</applyOffset>
+		<broadcastTF>True</broadcastTF>
+	</plugin>
+</gazebo>
 </robot>

File: rbcar_description/robots/versions/rbcar_faster.urdf.xacro (robot description, xacro)
@@ -9,9 +9,9 @@
 	<xacro:include filename="$(find rbcar_description)/urdf/bases/rbcar_base.urdf.xacro" />
 	<!-- Import Robotnik CAR wheels -->
-	<xacro:include filename="$(find rbcar_description)/urdf/wheels/suspension_wheel_v2.urdf.xacro" />
-	<xacro:include filename="$(find rbcar_description)/urdf/wheels/rear_axle.urdf.xacro" />
+	<xacro:include filename="$(find rbcar_description)/urdf/wheels/suspension_wheel_v3.urdf.xacro" />
 	<!-- Import all available sensors -->
 	<xacro:include filename="$(find rbcar_description)/urdf/structures/elevator.urdf.xacro" />
 	<xacro:include filename="$(find robotnik_sensors)/urdf/all_sensors.urdf.xacro" />
+  	<xacro:include filename="$(find robotnik_sensors)/urdf/utils/inertia.urdf.xacro" />
 	<!-- ***************** -->
 	<!-- Global parameters -->
@@ -19,12 +19,12 @@
 	<xacro:property name="PI" value="3.1415926535897931"/>
 	<!-- Wheel parameters -->
-	<xacro:property name="wheel_offset_x" value="1.0" />    <!-- x,y,z in translation from base_link to the center of the wheel -->
-	<xacro:property name="wheel_offset_y" value="0.75" />
+	<xacro:property name="wheel_offset_x" value="0.91131" />    <!-- x,y,z in translation from base_link to the center of the wheel -->
+	<xacro:property name="wheel_offset_y" value="0.62124" />
 	<xacro:property name="wheel_offset_z" value="0.0" />
 	<!-- Flag to select the high or low quality model -->
 	<xacro:property name="hq" value="true" />
 	<xacro:arg name="prefix" default="robot_"/>
-	<xacro:arg name="gps_longitude" default="39.5091874"/>
-	<xacro:arg name="gps_latitude" default="-0.4637371"/>
+	<xacro:arg name="gps_longitude" default="39.551218"/>
+	<xacro:arg name="gps_latitude" default="-0.467738"/>
 	<xacro:arg name="gpu" default="true"/>
 	<!-- *************** -->
@@ -32,20 +32,18 @@
 	<!-- *************** -->
 	<!-- Here we create the robot elements using the xacro:macros imported at the beggining of this file -->
+	<!-- Rbcar base -->
 	<xacro:rbcar_base name="rbcar" prefix="$(arg prefix)" publish_bf="true" hq="${hq}" />
 	<!-- Gazebo ros control pluggins -->
 	<xacro:ros_control/>
 	<!-- Wheels -->
-	<xacro:front_wheel lr_prefix="$(arg prefix)left" fr_prefix="front"
-					 lr_reflect="1" fr_reflect="1" parent="$(arg prefix)base_link" />
-	<xacro:front_wheel lr_prefix="$(arg prefix)right" fr_prefix="front"
-					 lr_reflect="-1" fr_reflect="1" parent="$(arg prefix)base_link" />
-	<xacro:rear_wheel lr_prefix="$(arg prefix)left" fr_prefix="rear"
-					lr_reflect="1" fr_reflect="-1" parent="$(arg prefix)base_link" />
-	<xacro:rear_wheel lr_prefix="$(arg prefix)right" fr_prefix="rear"
-					lr_reflect="-1" fr_reflect="-1" parent="$(arg prefix)base_link" />
-    <xacro:rear_axle prefix="$(arg prefix)rear_axle" parent="$(arg prefix)base_link">
-	  <origin xyz="0 0.0 0" rpy="1.57079633 0 3.14159265"/>
-    </xacro:rear_axle>
-	<!-- Sensors-->
+  	<xacro:front_wheel prefix="$(arg prefix)" lr_prefix="left" fr_prefix="front"
+                     lr_reflect="1" fr_reflect="1" parent="$(arg prefix)base_link" />
+  	<xacro:front_wheel prefix="$(arg prefix)" lr_prefix="right" fr_prefix="front"
+                     lr_reflect="-1" fr_reflect="1" parent="$(arg prefix)base_link" />
+  	<xacro:rear_wheel prefix="$(arg prefix)" lr_prefix="left" fr_prefix="rear"
+                    lr_reflect="1" fr_reflect="-1" parent="$(arg prefix)base_link" />
+  	<xacro:rear_wheel prefix="$(arg prefix)" lr_prefix="right" fr_prefix="rear"
+                    lr_reflect="-1" fr_reflect="-1" parent="$(arg prefix)base_link" />
+	<!-- SENSORS -->
 	<xacro:elevator parent="$(arg prefix)base_link" prefix="$(arg prefix)">
 		<origin xyz="0.0 0.0 0.6" rpy="0 0 0"/>
@@ -54,11 +52,11 @@
 		<origin xyz="0 0 0" rpy="0 0 0"/>
 	</xacro:sensor_axis_q8641>
-	<xacro:sensor_rslidar_16 prefix="$(arg prefix)top_3d_laser" parent="$(arg prefix)base_link" gpu="$(arg gpu)">
+	<xacro:sensor_rslidar_16 prefix="$(arg prefix)top_3d_laser" parent="$(arg prefix)base_link" gpu="$(arg gpu)"  prefix_topic="top_3d_laser">
 	  <origin xyz="1.39477 0.0 1.66733" rpy="0 0.673132 0"/> <!--rpy="0 0.261799 0" -->
 	</xacro:sensor_rslidar_16>
 	<!--M1-->
-	<xacro:sensor_hokuyo_utm30lx prefix="$(arg prefix)front_3d_laser" parent="$(arg prefix)base_link" gpu="$(arg gpu)">
+	<xacro:sensor_benewake_ce30d prefix="$(arg prefix)front_3d_laser" parent="$(arg prefix)base_link" gpu="$(arg gpu)" prefix_topic="front_3d_laser">
 	  <origin xyz="2.155 0.0 0.186" rpy="0 0.026 0"/>
-	</xacro:sensor_hokuyo_utm30lx>
+	</xacro:sensor_benewake_ce30d>
 	<xacro:sensor_imu_hector prefix="$(arg prefix)imu" parent="$(arg prefix)base_link">
 		<origin xyz="0.319 0.018 0.676" rpy="0 0 0"/>
@@ -71,5 +69,5 @@
   	</xacro:sensor_rubedos_viper>
 	<!--Hokuyo UTM30-->
-	<xacro:sensor_hokuyo_utm30lx prefix="$(arg prefix)front_laser" parent="$(arg prefix)base_link" gpu="$(arg gpu)">
+	<xacro:sensor_hokuyo_utm30lx prefix="$(arg prefix)front_laser" parent="$(arg prefix)base_link" gpu="$(arg gpu)" prefix_topic="front_laser">
 	  <origin xyz="1.289 0.0 1.364" rpy="0 0.0 0.0"/>
 	</xacro:sensor_hokuyo_utm30lx>

File: rbcar_description/robots/versions/rbcar_roborder.urdf.xacro (robot description, xacro)
@@ -1,4 +1,4 @@
 <?xml version="1.0"?>
-  <robot name="roborder"
+  <robot name="rbcar"
     xmlns:xacro="http://wiki.ros.org/xacro">
 	<!-- ***************** -->
@@ -10,6 +10,6 @@
 	<!-- Import Robotnik CAR wheels -->
 	<xacro:include filename="$(find rbcar_description)/urdf/wheels/suspension_wheel_v3.urdf.xacro" />
-	<xacro:include filename="$(find rbcar_description)/urdf/structures/elevator.urdf.xacro" />
 	<!-- Import all available sensors -->
+  <xacro:include filename="$(find rbcar_description)/urdf/structures/elevator.urdf.xacro" />
 	<xacro:include filename="$(find robotnik_sensors)/urdf/all_sensors.urdf.xacro" />
   <xacro:include filename="$(find robotnik_sensors)/urdf/utils/inertia.urdf.xacro" />
@@ -25,6 +25,6 @@
 	<xacro:property name="hq" value="true" />
         <xacro:arg name="prefix" default="robot_"/>
-        <xacro:arg name="gps_longitude" default="39.5091874"/>
-        <xacro:arg name="gps_latitude" default="-0.4637371"/>
+        <xacro:arg name="gps_longitude" default="39.551218"/>
+        <xacro:arg name="gps_latitude" default="-0.467738"/>
         <xacro:arg name="gpu" default="true"/>
 	<!-- *************** -->
@@ -32,20 +32,16 @@
 	<!-- *************** -->
 	<!-- Here we create the robot elements using the xacro:macros imported at the beggining of this file -->
-	<!-- Summit XL base -->
-	<xacro:rbcar_base name="roborder" prefix="$(arg prefix)" publish_bf="true" hq="${hq}" />
+	<!-- Rbcar base -->
+	<xacro:rbcar_base name="rbcar" prefix="$(arg prefix)" publish_bf="true" hq="${hq}" />
 	<!-- Gazebo ros control pluggins -->
 	<xacro:ros_control/>
-  <!-- xacro:omni_steering prefix="" publish_tf="true"/-->
-	<!-- Gazebo skid steering pluggins -->
-	<!-- xacro:skid_steering broadcastOdomTF="1"/ -->
-	<!-- WHEELS -->
   <!-- Wheels -->
-  <xacro:front_wheel lr_prefix="$(arg prefix)left" fr_prefix="front"
+  <xacro:front_wheel prefix="$(arg prefix)" lr_prefix="left" fr_prefix="front"
                      lr_reflect="1" fr_reflect="1" parent="$(arg prefix)base_link" />
-  <xacro:front_wheel lr_prefix="$(arg prefix)right" fr_prefix="front"
+  <xacro:front_wheel prefix="$(arg prefix)" lr_prefix="right" fr_prefix="front"
                      lr_reflect="-1" fr_reflect="1" parent="$(arg prefix)base_link" />
-  <xacro:rear_wheel lr_prefix="$(arg prefix)left" fr_prefix="rear"
+  <xacro:rear_wheel prefix="$(arg prefix)" lr_prefix="left" fr_prefix="rear"
                     lr_reflect="1" fr_reflect="-1" parent="$(arg prefix)base_link" />
-  <xacro:rear_wheel lr_prefix="$(arg prefix)right" fr_prefix="rear"
+  <xacro:rear_wheel prefix="$(arg prefix)" lr_prefix="right" fr_prefix="rear"
                     lr_reflect="-1" fr_reflect="-1" parent="$(arg prefix)base_link" />
 	<!-- SENSORS -->
@@ -56,4 +52,10 @@
       <origin xyz="1.289 0.0 1.354" rpy="0 0.0 0.0"/>
   </xacro:sensor_rubedos_viper>
+  <xacro:elevator parent="$(arg prefix)base_link" prefix="$(arg prefix)">
+		<origin xyz="0.0 0.0 0.6" rpy="0 0 0"/>
+	</xacro:elevator>
+	<xacro:sensor_axis_q8641 prefix="$(arg prefix)front_ptz_camera" parent="$(arg prefix)elevator_link" far="300" near="0.08">
+		<origin xyz="0 0 0" rpy="0 0 0"/>
+	</xacro:sensor_axis_q8641>
 	<xacro:sensor_imu_hector prefix="$(arg prefix)imu" parent="$(arg prefix)base_link">
 		<origin xyz="0.0 0.0 0.170" rpy="0 0 0"/>
@@ -62,10 +64,5 @@
 		<origin xyz="0.0 0 1.5" rpy="0 0 0"/>
 	</xacro:sensor_gps>
-  <xacro:elevator parent="$(arg prefix)base_link" prefix="$(arg prefix)">
-		<origin xyz="0.0 0.0 0.6" rpy="0 0 0"/>
-	</xacro:elevator>
-  <xacro:sensor_axis_q8641 prefix="$(arg prefix)front_ptz_camera" parent="$(arg prefix)elevator_link" far="300" near="0.08">
-    <origin xyz="0 0 0" rpy="0 0 0"/>
-  </xacro:sensor_axis_q8641>
+<!--Gazebo plugins-->
 <gazebo>
 <plugin name="ground_truth_controller" filename="librobotnik_gazebo_ground_truth_odom.so">

Commit message: Fix error in the model: The laser was rotate

File: rbcar_description/robots/rbcar.urdf.xacro (robot description, xacro)
@@ -53,5 +53,5 @@
 	</xacro:sensor_imu_hector>
 	<xacro:sensor_sick_outdoorscan3 prefix="$(arg prefix)front_laser" parent="$(arg prefix)base_link" prefix_topic="front_laser" min_angle="-1.5" max_angle="1.5" gpu="$(arg gpu)">
-		<origin xyz="2.15679 0 0.05433" rpy="0 0 0"/>
+		<origin xyz="2.15679 0 0.05433" rpy="${PI} 0 0"/>
 	</xacro:sensor_sick_outdoorscan3>
 	<xacro:sensor_gps prefix="$(arg prefix)gps" parent="$(arg prefix)base_link" gps_latitude="$(arg gps_latitude)" gps_longitude="$(arg gps_longitude)">

Commit message: Update rbcar_description

File: rbcar_description/robots/rbcar.urdf.xacro (robot description, xacro)
@@ -31,5 +31,5 @@
 	<!-- *************** -->
 	<!-- Here we create the robot elements using the xacro:macros imported at the beggining of this file -->
-	<!-- Summit XL base -->
+	<!-- Rbcar base -->
 	<xacro:rbcar_base name="rbcar" prefix="$(arg prefix)" publish_bf="true" hq="${hq}" />
 	<!-- Gazebo ros control pluggins -->
@@ -56,4 +56,7 @@
 		<origin xyz="2.101 0 0.206" rpy="0 0 0"/>
 	</xacro:sensor_sick_outdoorscan3>
+	<xacro:sensor_hokuyo_utm30lx prefix="$(arg prefix)rear_laser" parent="$(arg prefix)base_link" gpu="$(arg gpu)" prefix_topic="rear_laser">
+      		<origin xyz="-0.42925 0.0 0.24674" rpy="0 0 ${PI}"/>
+  	</xacro:sensor_hokuyo_utm30lx>
 	<xacro:sensor_gps prefix="$(arg prefix)gps" parent="$(arg prefix)base_link" gps_latitude="$(arg gps_latitude)" gps_longitude="$(arg gps_longitude)">
 		<origin xyz="0.491 0 1.503" rpy="0 0 0"/>

Commit message: Fix inertial physics of the model

File: rbcar_description/robots/rbcar.urdf.xacro (robot description, xacro)
@@ -9,8 +9,8 @@
 	<xacro:include filename="$(find rbcar_description)/urdf/bases/rbcar_base.urdf.xacro" />
 	<!-- Import Robotnik CAR wheels -->
-	<xacro:include filename="$(find rbcar_description)/urdf/wheels/suspension_wheel_v2.urdf.xacro" />
-	<xacro:include filename="$(find rbcar_description)/urdf/wheels/rear_axle.urdf.xacro" />
+	<xacro:include filename="$(find rbcar_description)/urdf/wheels/suspension_wheel_v3.urdf.xacro" />
 	<!-- Import all available sensors -->
 	<xacro:include filename="$(find robotnik_sensors)/urdf/all_sensors.urdf.xacro" />
+  	<xacro:include filename="$(find robotnik_sensors)/urdf/utils/inertia.urdf.xacro" />
 	<!-- ***************** -->
 	<!-- Global parameters -->
@@ -18,12 +18,12 @@
 	<xacro:property name="PI" value="3.1415926535897931"/>
 	<!-- Wheel parameters -->
-	<xacro:property name="wheel_offset_x" value="1.0" />    <!-- x,y,z in translation from base_link to the center of the wheel -->
-	<xacro:property name="wheel_offset_y" value="0.75" />
+	<xacro:property name="wheel_offset_x" value="0.91131" />    <!-- x,y,z in translation from base_link to the center of the wheel -->
+	<xacro:property name="wheel_offset_y" value="0.62124" />
 	<xacro:property name="wheel_offset_z" value="0.0" />
 	<!-- Flag to select the high or low quality model -->
 	<xacro:property name="hq" value="true" />
 	<xacro:arg name="prefix" default="robot_"/>
-	<xacro:arg name="gps_longitude" default="39.5091874"/>
-	<xacro:arg name="gps_latitude" default="-0.4637371"/>
+	<xacro:arg name="gps_longitude" default="39.551218"/>
+	<xacro:arg name="gps_latitude" default="-0.467738"/>
 	<xacro:arg name="gpu" default="true"/>
 	<!-- *************** -->
@@ -36,15 +36,12 @@
 	<xacro:ros_control/>
 	<!-- Wheels -->
-	<xacro:front_wheel lr_prefix="$(arg prefix)left" fr_prefix="front"
-					 lr_reflect="1" fr_reflect="1" parent="$(arg prefix)base_link" />
-	<xacro:front_wheel lr_prefix="$(arg prefix)right" fr_prefix="front"
-					 lr_reflect="-1" fr_reflect="1" parent="$(arg prefix)base_link" />
-	<xacro:rear_wheel lr_prefix="$(arg prefix)left" fr_prefix="rear"
-					lr_reflect="1" fr_reflect="-1" parent="$(arg prefix)base_link" />
-	<xacro:rear_wheel lr_prefix="$(arg prefix)right" fr_prefix="rear"
-					lr_reflect="-1" fr_reflect="-1" parent="$(arg prefix)base_link" />
-    <xacro:rear_axle prefix="$(arg prefix)rear_axle" parent="$(arg prefix)base_link">
-	  <origin xyz="0 0.0 0" rpy="1.57079633 0 3.14159265"/>
-    </xacro:rear_axle>
+  	<xacro:front_wheel prefix="$(arg prefix)" lr_prefix="left" fr_prefix="front"
+                     lr_reflect="1" fr_reflect="1" parent="$(arg prefix)base_link" />
+  	<xacro:front_wheel prefix="$(arg prefix)" lr_prefix="right" fr_prefix="front"
+                     lr_reflect="-1" fr_reflect="1" parent="$(arg prefix)base_link" />
+  	<xacro:rear_wheel prefix="$(arg prefix)" lr_prefix="left" fr_prefix="rear"
+                    lr_reflect="1" fr_reflect="-1" parent="$(arg prefix)base_link" />
+  	<xacro:rear_wheel prefix="$(arg prefix)" lr_prefix="right" fr_prefix="rear"
+                    lr_reflect="-1" fr_reflect="-1" parent="$(arg prefix)base_link" />
 	<xacro:sensor_rslidar_16 prefix="$(arg prefix)top_3d_laser" parent="$(arg prefix)base_link"  gpu="$(arg gpu)">
 	  <origin xyz="1.163 0.0 1.602" rpy="0 0.2637 0"/>
@@ -62,3 +59,36 @@
 		<origin xyz="0.491 0 1.503" rpy="0 0 0"/>
 	</xacro:sensor_gps>
+<!--Gazebo plugins-->
+<gazebo>
+	<plugin name="ground_truth_controller" filename="librobotnik_gazebo_ground_truth_odom.so">
+		<alwaysOn>true</alwaysOn>
+		<updateRate>50.0</updateRate>
+		<bodyName>$(arg prefix)base_link</bodyName>
+		<frameName>base_footprint_gt</frameName>
+		<worldBodyName>world</worldBodyName>
+		<worldFrameName>$(arg prefix)odom</worldFrameName>
+		<topicName>odom_gt</topicName>
+		<gaussianNoise>0.01</gaussianNoise>
+		<xyzOffset>0.0 0 0</xyzOffset>
+		<rpyOffset>0 0 0</rpyOffset>
+		<applyOffset>False</applyOffset>
+		<broadcastTF>True</broadcastTF>
+	</plugin>
+</gazebo>
+<gazebo>
+	<plugin name="gps_ground_truth_controller" filename="librobotnik_gazebo_ground_truth_odom.so">
+		<alwaysOn>true</alwaysOn>
+		<updateRate>50.0</updateRate>
+		<bodyName>$(arg prefix)gps_base_link</bodyName>
+		<frameName>gps_base_link_gt</frameName>
+		<worldBodyName>world</worldBodyName>
+		<worldFrameName>world</worldFrameName>
+		<topicName>odom_gt</topicName>
+		<gaussianNoise>0.01</gaussianNoise>
+		<xyzOffset>0.0 0 0</xyzOffset>
+		<rpyOffset>0 0 0</rpyOffset>
+		<applyOffset>False</applyOffset>
+		<broadcastTF>True</broadcastTF>
+	</plugin>
+</gazebo>
 </robot>
