Commit message: added fix from thecontruct repo

File: rbcar_description/robots/rbcar.urdf.xacro (robot description, xacro)
@@ -9,8 +9,8 @@
 	<xacro:include filename="$(find rbcar_description)/urdf/bases/rbcar_base.urdf.xacro" />
 	<!-- Import Robotnik CAR wheels -->
-	<xacro:include filename="$(find rbcar_description)/urdf/wheels/suspension_wheel_v3.urdf.xacro" />
+	<xacro:include filename="$(find rbcar_description)/urdf/wheels/suspension_wheel_v2.urdf.xacro" />
+	<xacro:include filename="$(find rbcar_description)/urdf/wheels/rear_axle.urdf.xacro" />
 	<!-- Import all available sensors -->
 	<xacro:include filename="$(find robotnik_sensors)/urdf/all_sensors.urdf.xacro" />
-  	<xacro:include filename="$(find robotnik_sensors)/urdf/utils/inertia.urdf.xacro" />
 	<!-- ***************** -->
 	<!-- Global parameters -->
@@ -18,31 +18,33 @@
 	<xacro:property name="PI" value="3.1415926535897931"/>
 	<!-- Wheel parameters -->
-	<xacro:property name="wheel_offset_x" value="0.91131" />    <!-- x,y,z in translation from base_link to the center of the wheel -->
-	<xacro:property name="wheel_offset_y" value="0.62124" />
+	<xacro:property name="wheel_offset_x" value="1.0" />    <!-- x,y,z in translation from base_link to the center of the wheel -->
+	<xacro:property name="wheel_offset_y" value="0.75" />
 	<xacro:property name="wheel_offset_z" value="0.0" />
 	<!-- Flag to select the high or low quality model -->
 	<xacro:property name="hq" value="true" />
 	<xacro:arg name="prefix" default="robot_"/>
-	<xacro:arg name="gps_longitude" default="39.551218"/>
-	<xacro:arg name="gps_latitude" default="-0.467738"/>
-	<xacro:arg name="gpu" default="true"/>
+	<xacro:arg name="gps_longitude" default="39.5091874"/>
+	<xacro:arg name="gps_latitude" default="-0.4637371"/>
 	<!-- *************** -->
 	<!-- Robots Elements -->
 	<!-- *************** -->
 	<!-- Here we create the robot elements using the xacro:macros imported at the beggining of this file -->
-	<!-- Rbcar base -->
+	<!-- Summit XL base -->
 	<xacro:rbcar_base name="rbcar" prefix="$(arg prefix)" publish_bf="true" hq="${hq}" />
 	<!-- Gazebo ros control pluggins -->
 	<xacro:ros_control/>
 	<!-- Wheels -->
-  	<xacro:front_wheel prefix="$(arg prefix)" lr_prefix="left" fr_prefix="front"
-                     lr_reflect="1" fr_reflect="1" parent="$(arg prefix)base_link" />
-  	<xacro:front_wheel prefix="$(arg prefix)" lr_prefix="right" fr_prefix="front"
-                     lr_reflect="-1" fr_reflect="1" parent="$(arg prefix)base_link" />
-  	<xacro:rear_wheel prefix="$(arg prefix)" lr_prefix="left" fr_prefix="rear"
-                    lr_reflect="1" fr_reflect="-1" parent="$(arg prefix)base_link" />
-  	<xacro:rear_wheel prefix="$(arg prefix)" lr_prefix="right" fr_prefix="rear"
-                    lr_reflect="-1" fr_reflect="-1" parent="$(arg prefix)base_link" />
-	<xacro:sensor_rslidar_16 prefix="$(arg prefix)top_3d_laser" parent="$(arg prefix)base_link"  gpu="$(arg gpu)">
+	<xacro:front_wheel lr_prefix="$(arg prefix)left" fr_prefix="front"
+					 lr_reflect="1" fr_reflect="1" parent="$(arg prefix)base_link" />
+	<xacro:front_wheel lr_prefix="$(arg prefix)right" fr_prefix="front"
+					 lr_reflect="-1" fr_reflect="1" parent="$(arg prefix)base_link" />
+	<xacro:rear_wheel lr_prefix="$(arg prefix)left" fr_prefix="rear"
+					lr_reflect="1" fr_reflect="-1" parent="$(arg prefix)base_link" />
+	<xacro:rear_wheel lr_prefix="$(arg prefix)right" fr_prefix="rear"
+					lr_reflect="-1" fr_reflect="-1" parent="$(arg prefix)base_link" />
+    <xacro:rear_axle prefix="$(arg prefix)rear_axle" parent="$(arg prefix)base_link">
+	  <origin xyz="0 0.0 0" rpy="1.57079633 0 3.14159265"/>
+    </xacro:rear_axle>
+	<xacro:sensor_rslidar_16 prefix="$(arg prefix)top_3d_laser" parent="$(arg prefix)base_link">
 	  <origin xyz="1.163 0.0 1.602" rpy="0 0.2637 0"/>
 	</xacro:sensor_rslidar_16>
@@ -50,45 +52,9 @@
 		<origin xyz="0.319 0.018 0.676" rpy="0 0 0"/>
 	</xacro:sensor_imu_hector>
-	<xacro:sensor_sick_outdoorscan3 prefix="$(arg prefix)front_laser" parent="$(arg prefix)base_link" prefix_topic="front_laser" min_angle="-1.5" max_angle="1.5" gpu="$(arg gpu)">
+	<xacro:sensor_sick_outdoorscan3 prefix="$(arg prefix)front_laser" parent="$(arg prefix)base_link" prefix_topic="front_laser" min_angle="-1.5" max_angle="1.5" gpu="false">
 		<origin xyz="2.101 0 0.206" rpy="0 0 0"/>
 	</xacro:sensor_sick_outdoorscan3>
-	<xacro:sensor_hokuyo_utm30lx prefix="$(arg prefix)rear_laser" parent="$(arg prefix)base_link" gpu="$(arg gpu)" prefix_topic="rear_laser">
-      		<origin xyz="-0.42925 0.0 0.24674" rpy="0 0 ${PI}"/>
-  	</xacro:sensor_hokuyo_utm30lx>
 	<xacro:sensor_gps prefix="$(arg prefix)gps" parent="$(arg prefix)base_link" gps_latitude="$(arg gps_latitude)" gps_longitude="$(arg gps_longitude)">
 		<origin xyz="0.491 0 1.503" rpy="0 0 0"/>
 	</xacro:sensor_gps>
-<!--Gazebo plugins-->
-<gazebo>
-	<plugin name="ground_truth_controller" filename="librobotnik_gazebo_ground_truth_odom.so">
-		<alwaysOn>true</alwaysOn>
-		<updateRate>50.0</updateRate>
-		<bodyName>$(arg prefix)base_link</bodyName>
-		<frameName>base_footprint_gt</frameName>
-		<worldBodyName>world</worldBodyName>
-		<worldFrameName>$(arg prefix)odom</worldFrameName>
-		<topicName>odom_gt</topicName>
-		<gaussianNoise>0.01</gaussianNoise>
-		<xyzOffset>0.0 0 0</xyzOffset>
-		<rpyOffset>0 0 0</rpyOffset>
-		<applyOffset>False</applyOffset>
-		<broadcastTF>True</broadcastTF>
-	</plugin>
-</gazebo>
-<gazebo>
-	<plugin name="gps_ground_truth_controller" filename="librobotnik_gazebo_ground_truth_odom.so">
-		<alwaysOn>true</alwaysOn>
-		<updateRate>50.0</updateRate>
-		<bodyName>$(arg prefix)gps_base_link</bodyName>
-		<frameName>gps_base_link_gt</frameName>
-		<worldBodyName>world</worldBodyName>
-		<worldFrameName>world</worldFrameName>
-		<topicName>odom_gt</topicName>
-		<gaussianNoise>0.01</gaussianNoise>
-		<xyzOffset>0.0 0 0</xyzOffset>
-		<rpyOffset>0 0 0</rpyOffset>
-		<applyOffset>False</applyOffset>
-		<broadcastTF>True</broadcastTF>
-	</plugin>
-</gazebo>
 </robot>

File: rbcar_description/urdf/wheels/suspension_wheel_v3.urdf.xacro (robot description, xacro)
@@ -7,7 +7,7 @@
        axle_length. -->
   <xacro:property name="hub_dia" value="0.235"/>
-  <xacro:property name="tire_dia" value="0.639"/>
-  <xacro:property name="tire_width" value="0.245"/>
-  <xacro:property name="hex_hub_depth" value="0.0"/> <!-- or +0.072 -->
+  <xacro:property name="tire_dia" value="0.634"/>
+  <xacro:property name="tire_width" value="0.322"/>
+  <xacro:property name="hex_hub_depth" value="0.120"/> <!-- or +0.072 -->
   <xacro:property name="wheel_mass" value="8.0"/>   <!-- check -->
   <!-- hex_hub_dist is the distance between left and right hex hubs when
@@ -17,6 +17,5 @@
   <xacro:property name="wheelbase" value="1.83323"/>
   <!--xacro:property name="hex_hub_dist" value="1.2385"/-->  <!-- 1.127 0.742 0.900 check -->
-  <!--xacro:property name="axle_length" value="0.120"/-->
-  <xacro:property name="axle_length" value="0.12"/>
+  <xacro:property name="axle_length" value="0.120"/>
   <xacro:property name="wheel_travel" value="0.1"/>
   <xacro:property name="shock_z_offset" value="0.05"/>
@@ -70,11 +69,11 @@
     <inertial>
       <mass value="0.001"/>
-      <inertia ixx="0.001" ixy="0" ixz="0" iyy="0.001" iyz="0" izz="0.001"/>
+      <inertia ixx="1.6666666666666666e-10" ixy="0" ixz="0" iyy="1.6666666666666666e-10" iyz="0" izz="1.6666666666666666e-10"/>
     </inertial>
   </xacro:macro>
   <!-- Shock absorber -->
   <xacro:macro name="shock"
-               params="prefix lr_prefix fr_prefix lr_reflect fr_reflect child parent">
-    <joint name="${prefix}${lr_prefix}_${fr_prefix}_shock" type="fixed">
+               params="lr_prefix fr_prefix lr_reflect fr_reflect child parent">
+    <joint name="${lr_prefix}_${fr_prefix}_shock" type="fixed">
       <parent link="${parent}"/>
       <child link="${child}"/>
@@ -90,16 +89,41 @@
                    ${lr_reflect * ((hex_hub_dist / 2) - axle_length )}
                    ${(wheel_travel / 2) - shock_z_offset}"/>
+      <!--axis xyz="0 0 -1"/-->
+      <!--limit lower="${-wheel_travel / 2}" upper="${wheel_travel / 2}"
+             effort="${shock_eff_limit}" velocity="${shock_vel_limit}"/>
+      <joint_properties damping="${suspension_joint_damping}" friction="${suspension_joint_friction}"/-->
     </joint>
+    <!--transmission name="${lr_prefix}_${fr_prefix}_shock_trans">
+      <type>transmission_interface/SimpleTransmission</type>
+      <joint name="${lr_prefix}_${fr_prefix}_shock">
+        <hardwareInterface>hardware_interface/EffortJointInterface</hardwareInterface>
+      </joint>
+      <actuator name="${lr_prefix}_${fr_prefix}_shock_act">
+        <mechanicalReduction>1</mechanicalReduction>
+      </actuator>
+    </transmission-->
   </xacro:macro>
   <!-- The "wheel" macro defines an axle carrier, axle, and wheel. -->
-  <xacro:macro name="wheel" params="prefix lr_prefix fr_prefix lr_reflect">
-    <link name="${prefix}${lr_prefix}_${fr_prefix}_axle_carrier">
+  <xacro:macro name="wheel" params="lr_prefix fr_prefix lr_reflect ackerman_debug:=0">
+    <link name="${lr_prefix}_${fr_prefix}_axle_carrier">
+	  <!-- visual>
+        <origin xyz="0 0 0"/>
+        <geometry>
+          <cylinder radius="0.1" length="0.1"/>
+        </geometry>
+	  </visual>
+	  <collision>
+        <origin xyz="0 0 0"/>
+        <geometry>
+          <cylinder radius="0.1" length="0.1"/>
+        </geometry>
+	  </collision -->
       <xacro:null_inertial/>
     </link>
     <!-- The left and right axles have the same axis so that identical
          rotation values cause the wheels to rotate in the same direction. -->
-    <joint name="${prefix}${lr_prefix}_${fr_prefix}_axle" type="continuous">
-      <parent link="${prefix}${lr_prefix}_${fr_prefix}_axle_carrier"/>
-      <child link="${prefix}${lr_prefix}_${fr_prefix}_wheel"/>
+    <joint name="${lr_prefix}_${fr_prefix}_axle" type="continuous">
+      <parent link="${lr_prefix}_${fr_prefix}_axle_carrier"/>
+      <child link="${lr_prefix}_${fr_prefix}_wheel"/>
       <origin rpy="${degrees_90} 0 ${degrees_180}"/>
       <axis xyz="0 0 1"/>
@@ -107,28 +131,28 @@
       <joint_properties damping="${wheel_joint_damping}" friction="${wheel_joint_friction}"/>
     </joint>
-    <transmission name="${prefix}${lr_prefix}_${fr_prefix}_axle_trans">
+    <transmission name="${lr_prefix}_${fr_prefix}_axle_trans">
       <type>transmission_interface/SimpleTransmission</type>
-      <joint name="${prefix}${lr_prefix}_${fr_prefix}_axle">
-        <!-- hardwareInterface>hardware_interface/EffortJointInterface</hardwareInterface -->
-        <hardwareInterface>hardware_interface/VelocityJointInterface</hardwareInterface>
-      </joint>
-      <actuator name="${prefix}${lr_prefix}_${fr_prefix}_axle_act">
+      <joint name="${lr_prefix}_${fr_prefix}_axle">
+        <hardwareInterface>hardware_interface/EffortJointInterface</hardwareInterface>
+        <!-- <hardwareInterface>hardware_interface/VelocityJointInterface</hardwareInterface> -->
+      </joint>
+      <actuator name="${lr_prefix}_${fr_prefix}_axle_act">
         <mechanicalReduction>1</mechanicalReduction>
       </actuator>
     </transmission>
-    <gazebo reference="${prefix}${lr_prefix}_${fr_prefix}_axle_carrier">
+    <gazebo reference="${lr_prefix}_${fr_prefix}_axle_carrier">
       <material>Gazebo/Black</material>
     </gazebo>
-    <link name="${prefix}${lr_prefix}_${fr_prefix}_wheel">
+    <link name="${lr_prefix}_${fr_prefix}_wheel">
       <visual>
         <xacro:if value="${lr_prefix=='left'}">
           <origin xyz="0
                        0
-                       ${lr_reflect * (axle_length - (tire_width / 2 - hex_hub_depth)) - 0.08} " rpy = "-${degrees_90} 0 ${degrees_180}"/>
+                       ${lr_reflect * (axle_length - (tire_width / 2 - hex_hub_depth))}" rpy = "${degrees_90} 0 ${degrees_180}"/>
         </xacro:if>
         <xacro:if value="${lr_prefix=='right'}">
           <origin xyz="0
                        0
-                       ${lr_reflect * (axle_length - (tire_width / 2 - hex_hub_depth)) + 0.08} " rpy = "${degrees_90} 0 ${degrees_180}"/>
+                       ${lr_reflect * (axle_length - (tire_width / 2 - hex_hub_depth))}" rpy = "-${degrees_90} 0 ${degrees_180}"/>
         </xacro:if>
         <geometry>
@@ -150,16 +174,32 @@
           height="${tire_width}" mass="${wheel_mass}"/>
     </link>
-    <gazebo reference="${prefix}${lr_prefix}_${fr_prefix}_wheel">
+    <gazebo reference="${lr_prefix}_${fr_prefix}_wheel">
       <material>Gazebo/Black</material>
     </gazebo>
+    <!-- Visualization Ackerman -->
+    <xacro:if value="${ackerman_debug == 1}"> <!-- this applies if we are setting the left wheel -->
+      <link name="${lr_prefix}_${fr_prefix}_wheel_axis">
+        <visual>
+          <origin xyz="0 0 0" rpy = "0 0 0"/>
+          <geometry>
+            <cylinder radius="0.05" length="10.0"/>
+          </geometry>
+          <material name="tire_mat"/>
+        </visual>
+      </link>
+      <joint name="${lr_prefix}_${fr_prefix}_ackerman_joint" type="fixed">
+        <parent link="${lr_prefix}_${fr_prefix}_wheel"/>
+        <child link="${lr_prefix}_${fr_prefix}_wheel_axis"/>
+      </joint>
+    </xacro:if>
   </xacro:macro>
   <!-- xacro:macro name="rubber_wheel" params="name parent *origin reflect hq" -->
   <!-- Front wheel -->
   <xacro:macro name="front_wheel"
-               params="prefix lr_prefix fr_prefix lr_reflect fr_reflect parent">
-    <xacro:shock prefix="${prefix}" lr_prefix="${lr_prefix}" fr_prefix="${fr_prefix}"
+               params="lr_prefix fr_prefix lr_reflect fr_reflect parent">
+    <xacro:shock lr_prefix="${lr_prefix}" fr_prefix="${fr_prefix}"
                  lr_reflect="${lr_reflect}" fr_reflect="${fr_reflect}"
-                 child="${prefix}${lr_prefix}_steering_link" parent="${parent}"/>
-    <link name="${prefix}${lr_prefix}_steering_link">
+                 child="${lr_prefix}_steering_link" parent="${parent}"/>
+    <link name="${lr_prefix}_steering_link">
 	  <!-- visual>
 		<origin xyz="0 0 0"/>
@@ -176,7 +216,7 @@
       <xacro:null_inertial/>
     </link>
-    <joint name="${prefix}${lr_prefix}_steering_joint" type="revolute">
-      <parent link="${prefix}${lr_prefix}_steering_link"/>
-      <child link="${prefix}${lr_prefix}_${fr_prefix}_axle_carrier"/>
+    <joint name="${lr_prefix}_steering_joint" type="revolute">
+      <parent link="${lr_prefix}_steering_link"/>
+      <child link="${lr_prefix}_${fr_prefix}_axle_carrier"/>
       <axis xyz="0 0 1"/>
       <xacro:if value="${lr_reflect == 1}"> <!-- this applies if we are setting the left wheel -->
@@ -189,27 +229,27 @@
       </xacro:unless>
     </joint>
-    <transmission name="${prefix}${lr_prefix}_steering_trans">
+    <transmission name="${lr_prefix}_steering_trans">
       <type>transmission_interface/SimpleTransmission</type>
-      <joint name="${prefix}${lr_prefix}_steering_joint">
-        <!--<hardwareInterface>hardware_interface/EffortJointInterface</hardwareInterface>-->
-        <hardwareInterface>hardware_interface/PositionJointInterface</hardwareInterface>
-      </joint>
-      <actuator name="${prefix}${lr_prefix}_steering_act">
+      <joint name="${lr_prefix}_steering_joint">
+        <hardwareInterface>hardware_interface/EffortJointInterface</hardwareInterface>
+        <!-- <hardwareInterface>hardware_interface/PositionJointInterface</hardwareInterface> -->
+      </joint>
+      <actuator name="${lr_prefix}_steering_act">
         <mechanicalReduction>1</mechanicalReduction>
       </actuator>
     </transmission>
-    <gazebo reference="${prefix}${lr_prefix}_steering_link">
+    <gazebo reference="${lr_prefix}_steering_link">
       <material>Gazebo/Black</material>
     </gazebo>
-    <xacro:wheel prefix="${prefix}" lr_prefix="${lr_prefix}" fr_prefix="${fr_prefix}"
+    <xacro:wheel lr_prefix="${lr_prefix}" fr_prefix="${fr_prefix}"
                  lr_reflect="${lr_reflect}"/>
   </xacro:macro>
   <!-- Rear wheel -->
   <xacro:macro name="rear_wheel"
-               params="prefix lr_prefix fr_prefix lr_reflect fr_reflect parent">
-    <xacro:shock prefix="${prefix}" lr_prefix="${lr_prefix}" fr_prefix="${fr_prefix}"
+               params="lr_prefix fr_prefix lr_reflect fr_reflect parent">
+    <xacro:shock lr_prefix="${lr_prefix}" fr_prefix="${fr_prefix}"
                  lr_reflect="${lr_reflect}" fr_reflect="${fr_reflect}"
-                 child="${prefix}${lr_prefix}_${fr_prefix}_axle_carrier" parent="${parent}"/>
-    <xacro:wheel prefix="${prefix}" lr_prefix="${lr_prefix}" fr_prefix="${fr_prefix}"
+                 child="${lr_prefix}_${fr_prefix}_axle_carrier" parent="${parent}"/>
+    <xacro:wheel lr_prefix="${lr_prefix}" fr_prefix="${fr_prefix}"
                  lr_reflect="${lr_reflect}"/>
   </xacro:macro>
