Commit message: Update position of gps

File: rbcar_description/robots/versions/rbcar_faster.urdf.xacro (robot description, xacro)
@@ -64,5 +64,5 @@
 	</xacro:sensor_imu_hector>
 	<xacro:sensor_gps prefix="$(arg prefix)gps" parent="$(arg prefix)base_link" gps_latitude="$(arg gps_latitude)" gps_longitude="$(arg gps_longitude)">
-		<origin xyz="0.491 0 1.503" rpy="0 0 0"/>
+		<origin xyz="0.491 -0.5272 1.503" rpy="0 0 0"/>
 	</xacro:sensor_gps>
 	<xacro:sensor_rubedos_viper prefix="$(arg prefix)viper" parent="$(arg prefix)base_link">

Commit message: viper x position from 0.6 to 1.289

File: rbcar_description/robots/versions/rbcar_faster.urdf.xacro (robot description, xacro)
@@ -67,5 +67,5 @@
 	</xacro:sensor_gps>
 	<xacro:sensor_rubedos_viper prefix="$(arg prefix)viper" parent="$(arg prefix)base_link">
-      <origin xyz="0.6 0.0 1.354" rpy="0 0.1745 0.0"/>
+      <origin xyz="1.289 0.0 1.354" rpy="0 0.1745 0.0"/>
   	</xacro:sensor_rubedos_viper>
 <!--Gazebo plugins-->

Commit message: Update urdf rbcar_faster

File: rbcar_description/robots/versions/rbcar_faster.urdf.xacro (robot description, xacro)
@@ -55,8 +55,9 @@
 	</xacro:sensor_axis_q8641>
 	<xacro:sensor_rslidar_16 prefix="$(arg prefix)top_3d_laser" parent="$(arg prefix)base_link" gpu="$(arg gpu)">
-	  <origin xyz="1.39477 0.0 2.07733" rpy="0 0.698132 0"/> <!--rpy="0 0.261799 0" -->
+	  <origin xyz="1.39477 0.0 1.66733" rpy="0 0.673132 0"/> <!--rpy="0 0.261799 0" -->
 	</xacro:sensor_rslidar_16>
+	<!--M1-->
 	<xacro:sensor_hokuyo_utm30lx prefix="$(arg prefix)front_3d_laser" parent="$(arg prefix)base_link" gpu="$(arg gpu)">
-	  <origin xyz="2.155 0.0 0.236" rpy="0 0 0"/>
+	  <origin xyz="2.155 0.0 0.186" rpy="0 0.026 0"/>
 	</xacro:sensor_hokuyo_utm30lx>
 	<xacro:sensor_imu_hector prefix="$(arg prefix)imu" parent="$(arg prefix)base_link">
@@ -67,6 +68,10 @@
 	</xacro:sensor_gps>
 	<xacro:sensor_rubedos_viper prefix="$(arg prefix)viper" parent="$(arg prefix)base_link">
-      <origin xyz="1.289 0.0 1.354" rpy="0 0.1745 0.0"/>
+      <origin xyz="1.289 0.0 1.354" rpy="0 0.0 0.0"/>
   	</xacro:sensor_rubedos_viper>
+	<!--Hokuyo UTM30-->
+	<xacro:sensor_hokuyo_utm30lx prefix="$(arg prefix)front_laser" parent="$(arg prefix)base_link" gpu="$(arg gpu)">
+	  <origin xyz="1.289 0.0 1.364" rpy="0 0.0 0.0"/>
+	</xacro:sensor_hokuyo_utm30lx>
 <!--Gazebo plugins-->
 <gazebo>
