Commit message: axis model changed to axis_q8641

File: rbcar_description/robots/versions/rbcar_roborder.urdf.xacro (robot description, xacro)
@@ -46,8 +46,9 @@
 	<!-- SENSORS -->
     <xacro:sensor_benewake_ce30d prefix="front_3d_lidar" parent="base_link" gpu="true">
-        <origin xyz="2.155 0.0 0.236" rpy="0 0.24396 0"/>
+        <origin xyz="2.155 0.0 0.236" rpy="0 0 0"/>
     </xacro:sensor_benewake_ce30d>
     <xacro:sensor_rubedos_viper prefix="viper" parent="base_link">
-        <origin xyz="1.289 0.0 1.354" rpy="0 0.1745 0.0"/>
+        <!--origin xyz="1.289 0.0 1.354" rpy="0 0.1745 0.0"/-->
+        <origin xyz="1.289 0.0 1.354" rpy="0 0.0 0.0"/>
     </xacro:sensor_rubedos_viper>
 	<xacro:sensor_imu_hector prefix="imu" parent="base_link">
@@ -62,7 +63,7 @@
 		<origin xyz="0.0 0.0 0.6" rpy="0 0 0"/>
 	</xacro:elevator>
-    <xacro:sensor_axis prefix="front_ptz_camera" parent="elevator_link" far="300" near="0.08">
+    <xacro:sensor_axis_q8641 prefix="front_ptz_camera" parent="elevator_link" far="300" near="0.08">
             <origin xyz="0 0 0" rpy="0 0 0"/>
-    </xacro:sensor_axis>
+    </xacro:sensor_axis_q8641>
 <gazebo>
 <plugin name="ground_truth_controller" filename="librobotnik_gazebo_ground_truth_odom.so">

Commit message: fixed viper position and other things

File: rbcar_description/robots/versions/rbcar_roborder.urdf.xacro (robot description, xacro)
@@ -13,4 +13,5 @@
 	<!-- Import all available sensors -->
 	<xacro:include filename="$(find robotnik_sensors)/urdf/all_sensors.urdf.xacro" />
+  <xacro:include filename="$(find robotnik_sensors)/urdf/utils/inertia.urdf.xacro" />
 	<!-- ***************** -->
 	<!-- Global parameters -->
@@ -31,39 +32,36 @@
 	<!-- Gazebo ros control pluggins -->
 	<xacro:ros_control/>
-        <!-- xacro:omni_steering prefix="" publish_tf="true"/-->
+  <!-- xacro:omni_steering prefix="" publish_tf="true"/-->
 	<!-- Gazebo skid steering pluggins -->
 	<!-- xacro:skid_steering broadcastOdomTF="1"/ -->
 	<!-- WHEELS -->
-    <!-- Wheels -->
-    <xacro:front_wheel lr_prefix="left" fr_prefix="front"
-                       lr_reflect="1" fr_reflect="1" parent="base_link" />
-    <xacro:front_wheel lr_prefix="right" fr_prefix="front"
-                       lr_reflect="-1" fr_reflect="1" parent="base_link" />
-    <xacro:rear_wheel lr_prefix="left" fr_prefix="rear"
-                      lr_reflect="1" fr_reflect="-1" parent="base_link" />
-    <xacro:rear_wheel lr_prefix="right" fr_prefix="rear"
-                      lr_reflect="-1" fr_reflect="-1" parent="base_link" />
+  <!-- Wheels -->
+  <xacro:front_wheel lr_prefix="left" fr_prefix="front"
+                     lr_reflect="1" fr_reflect="1" parent="base_link" />
+  <xacro:front_wheel lr_prefix="right" fr_prefix="front"
+                     lr_reflect="-1" fr_reflect="1" parent="base_link" />
+  <xacro:rear_wheel lr_prefix="left" fr_prefix="rear"
+                    lr_reflect="1" fr_reflect="-1" parent="base_link" />
+  <xacro:rear_wheel lr_prefix="right" fr_prefix="rear"
+                    lr_reflect="-1" fr_reflect="-1" parent="base_link" />
 	<!-- SENSORS -->
-    <xacro:sensor_benewake_ce30d prefix="front_3d_lidar" parent="base_link" gpu="true">
-        <origin xyz="2.155 0.0 0.236" rpy="0 0 0"/>
-    </xacro:sensor_benewake_ce30d>
-    <xacro:sensor_rubedos_viper prefix="viper" parent="base_link">
-        <!--origin xyz="1.289 0.0 1.354" rpy="0 0.1745 0.0"/-->
-        <origin xyz="1.289 0.0 1.354" rpy="0 0.0 0.0"/>
-    </xacro:sensor_rubedos_viper>
+  <xacro:sensor_benewake_ce30d prefix="front_3d_lidar" parent="base_link" gpu="true">
+      <origin xyz="2.155 0.0 0.236" rpy="0 0 0"/>
+  </xacro:sensor_benewake_ce30d>
+  <xacro:sensor_rubedos_viper prefix="viper" parent="base_link">
+      <origin xyz="1.289 0.0 1.354" rpy="0 0.0 0.0"/>
+  </xacro:sensor_rubedos_viper>
 	<xacro:sensor_imu_hector prefix="imu" parent="base_link">
 		<origin xyz="0.0 0.0 0.170" rpy="0 0 0"/>
-		<!--<origin xyz="0.917 0.0 0.170" rpy="0 0 0"/>-->
 	</xacro:sensor_imu_hector>
 	<xacro:sensor_gps prefix="gps" parent="base_link" gps_latitude="$(arg gps_latitude)" gps_longitude="$(arg gps_longitude)" update_rate="20" >
 		<origin xyz="0.0 0 1.5" rpy="0 0 0"/>
-		<!--<origin xyz="0.747 0 1.5" rpy="0 0 0"/>-->
 	</xacro:sensor_gps>
-    <xacro:elevator parent="base_link">
+  <xacro:elevator parent="base_link">
 		<origin xyz="0.0 0.0 0.6" rpy="0 0 0"/>
 	</xacro:elevator>
-    <xacro:sensor_axis_q8641 prefix="front_ptz_camera" parent="elevator_link" far="300" near="0.08">
-            <origin xyz="0 0 0" rpy="0 0 0"/>
-    </xacro:sensor_axis_q8641>
+  <xacro:sensor_axis_q8641 prefix="front_ptz_camera" parent="elevator_link" far="300" near="0.08">
+    <origin xyz="0 0 0" rpy="0 0 0"/>
+  </xacro:sensor_axis_q8641>
 <gazebo>
 <plugin name="ground_truth_controller" filename="librobotnik_gazebo_ground_truth_odom.so">

Commit message: added new wheel model of polaris

File: rbcar_description/robots/versions/rbcar_roborder.urdf.xacro (robot description, xacro)
@@ -9,5 +9,5 @@
 	<xacro:include filename="$(find rbcar_description)/urdf/bases/rbcar_base.urdf.xacro" />
 	<!-- Import Robotnik CAR wheels -->
-	<xacro:include filename="$(find rbcar_description)/urdf/wheels/suspension_wheel_v2.urdf.xacro" />
+	<xacro:include filename="$(find rbcar_description)/urdf/wheels/suspension_wheel_v3.urdf.xacro" />
 	<xacro:include filename="$(find rbcar_description)/urdf/structures/elevator.urdf.xacro" />
 	<!-- Import all available sensors -->
@@ -19,6 +19,6 @@
 	<xacro:property name="PI" value="3.1415926535897931"/>
 	<!-- Wheel parameters -->
-	<xacro:property name="wheel_offset_x" value="1.0" />    <!-- x,y,z in translation from base_link to the center of the wheel -->
-	<xacro:property name="wheel_offset_y" value="0.75" />
+	<xacro:property name="wheel_offset_x" value="0.91131" />    <!-- x,y,z in translation from base_link to the center of the wheel -->
+	<xacro:property name="wheel_offset_y" value="0.62124" />
 	<xacro:property name="wheel_offset_z" value="0.0" />
 	<!-- Flag to select the high or low quality model -->

Commit message: Update description of robot

File: rbcar_description/robots/versions/rbcar_roborder.urdf.xacro (robot description, xacro)
@@ -25,5 +25,8 @@
 	<!-- Flag to select the high or low quality model -->
 	<xacro:property name="hq" value="true" />
-  <xacro:arg name="prefix" default="robot_"/>
+        <xacro:arg name="prefix" default="robot_"/>
+        <xacro:arg name="gps_longitude" default="39.5091874"/>
+        <xacro:arg name="gps_latitude" default="-0.4637371"/>
+        <xacro:arg name="gpu" default="true"/>
 	<!-- *************** -->
 	<!-- Robots Elements -->
@@ -48,10 +51,10 @@
                     lr_reflect="-1" fr_reflect="-1" parent="$(arg prefix)base_link" />
 	<!-- SENSORS -->
-  <xacro:sensor_benewake_ce30d prefix="$(arg prefix)front_3d_lidar" parent="$(arg prefix)base_link" gpu="true">
+  <!--xacro:sensor_benewake_ce30d prefix="$(arg prefix)front_3d_lidar" parent="$(arg prefix)base_link" gpu="$(arg gpu)">
       <origin xyz="2.155 0.0 0.236" rpy="0 0 0"/>
-  </xacro:sensor_benewake_ce30d>
-  <xacro:sensor_rubedos_viper prefix="$(arg prefix)viper" parent="$(arg prefix)base_link">
+  </xacro:sensor_benewake_ce30d-->
+  <!--xacro:sensor_rubedos_viper prefix="$(arg prefix)viper" parent="$(arg prefix)base_link">
       <origin xyz="1.289 0.0 1.354" rpy="0 0.0 0.0"/>
-  </xacro:sensor_rubedos_viper>
+  </xacro:sensor_rubedos_viper!-->
 	<xacro:sensor_imu_hector prefix="$(arg prefix)imu" parent="$(arg prefix)base_link">
 		<origin xyz="0.0 0.0 0.170" rpy="0 0 0"/>
@@ -66,4 +69,7 @@
     <origin xyz="0 0 0" rpy="0 0 0"/>
   </xacro:sensor_axis_q8641>
+  <!--xacro:sensor_rslidar_16 prefix="$(arg prefix)top_3d_laser" parent="$(arg prefix)base_link"  gpu="$(arg gpu)">
+    <origin xyz="1.163 0.0 1.602" rpy="0 0.2637 0"/>
+  </xacro:sensor_rslidar_16-->
 <gazebo>
 <plugin name="ground_truth_controller" filename="librobotnik_gazebo_ground_truth_odom.so">

File: rbcar_description/urdf/bases/roborder_base.urdf.xacro (robot description, xacro)
@@ -2,5 +2,5 @@
 <robot name="roborder" xmlns:xacro="http://wiki.ros.org/xacro">
   <xacro:include filename="$(find rbcar_description)/urdf/bases/roborder_base.gazebo.xacro" />
-  <xacro:macro name="roborder_base" params="name publish_bf hq">
+  <xacro:macro name="roborder_base" params="prefix:='' name publish_bf hq">
   <!-- Robot mechanical and motor parameters -->
   <xacro:property name="PI" value="3.1415926535897931"/>
@@ -10,5 +10,5 @@
   <!-- BASE FOOTPRINT -->
   <xacro:if value="${publish_bf}">
-    <link name="base_footprint">
+    <link name="${prefix}base_footprint">
       <visual>
           <origin xyz="0 0 0" rpy="0 0 0" />
@@ -26,12 +26,12 @@
 -->
     </link>
-    <joint name="base_footprint_joint" type="fixed">
+    <joint name="${prefix}base_footprint_joint" type="fixed">
       <origin xyz="0 0 ${clearance}" rpy="0 0 0" />  <!-- height is the clearance -->
-      <parent link="base_footprint"/>
-      <child link="base_link" />
+      <parent link="${prefix}base_footprint"/>
+      <child link="${prefix}base_link" />
     </joint>
   </xacro:if>
   <!-- BASE_LINK -->
-  <link name="base_link">
+  <link name="${prefix}base_link">
     <inertial>
       <mass value="125.0" />

Commit message: merge rbcar_faster to melodic-devel

File: rbcar_description/robots/versions/rbcar_roborder.urdf.xacro (robot description, xacro)
@@ -9,6 +9,5 @@
 	<xacro:include filename="$(find rbcar_description)/urdf/bases/rbcar_base.urdf.xacro" />
 	<!-- Import Robotnik CAR wheels -->
-	<!--xacro:include filename="$(find rbcar_description)/urdf/wheels/suspension_wheel_v3.urdf.xacro" /-->
-  <xacro:include filename="$(find rbcar_description)/urdf/wheels/suspension_wheel_v2.urdf.xacro" />
+	<xacro:include filename="$(find rbcar_description)/urdf/wheels/suspension_wheel_v3.urdf.xacro" />
 	<xacro:include filename="$(find rbcar_description)/urdf/structures/elevator.urdf.xacro" />
 	<!-- Import all available sensors -->
@@ -51,10 +50,10 @@
                     lr_reflect="-1" fr_reflect="-1" parent="$(arg prefix)base_link" />
 	<!-- SENSORS -->
-  <!--xacro:sensor_benewake_ce30d prefix="$(arg prefix)front_3d_lidar" parent="$(arg prefix)base_link" gpu="$(arg gpu)">
+  <xacro:sensor_benewake_ce30d prefix="$(arg prefix)front_3d_lidar" parent="$(arg prefix)base_link" gpu="$(arg gpu)">
       <origin xyz="2.155 0.0 0.236" rpy="0 0 0"/>
-  </xacro:sensor_benewake_ce30d-->
-  <!--xacro:sensor_rubedos_viper prefix="$(arg prefix)viper" parent="$(arg prefix)base_link">
+  </xacro:sensor_benewake_ce30d>
+  <xacro:sensor_rubedos_viper prefix="$(arg prefix)viper" parent="$(arg prefix)base_link">
       <origin xyz="1.289 0.0 1.354" rpy="0 0.0 0.0"/>
-  </xacro:sensor_rubedos_viper!-->
+  </xacro:sensor_rubedos_viper>
 	<xacro:sensor_imu_hector prefix="$(arg prefix)imu" parent="$(arg prefix)base_link">
 		<origin xyz="0.0 0.0 0.170" rpy="0 0 0"/>
@@ -69,7 +68,4 @@
     <origin xyz="0 0 0" rpy="0 0 0"/>
   </xacro:sensor_axis_q8641>
-  <!--xacro:sensor_rslidar_16 prefix="$(arg prefix)top_3d_laser" parent="$(arg prefix)base_link"  gpu="$(arg gpu)">
-    <origin xyz="1.163 0.0 1.602" rpy="0 0.2637 0"/>
-  </xacro:sensor_rslidar_16-->
 <gazebo>
 <plugin name="ground_truth_controller" filename="librobotnik_gazebo_ground_truth_odom.so">
